File: HW/GMWPY/GMWPY.kicad_sch (KiCad schematic)
At the start: 14 parts, among them U1 USEQGCDACH4100, U2 TSV991ILT, U3 TSV991ILT, U4 EC4-1000-H2

Commit message: g
Other:
- note added: "1.2 V, 0.1 A or 25 mW absolute max but in practice under 0.7v"
Changed lines of the file:
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@@
     (stroke (width 0) (type default) (color 0 0 0 0))
+  )
+  (text " 1.2 V, 0.1 A or 25 mW absolute max\nbut in practice under 0.7v"
+    (at 30.48 146.05 0)
+    (effects (font (size 1.27 1.27)) (justify left bottom))
   )
   (label "OUT2" (at 170.18 59.69 0)

Commit message: r
Parts:
- added C7, C8, C9, C?: 100n, Capacitor_SMD:C_0603_1608Metric, symbol Device:C_Small
- added Q1: Q_PJFET_DSG, Package_TO_SOT_SMD:SOT-23, symbol Device:Q_PJFET_DSG
- added R10, R6, R7: 10k, Resistor_SMD:R_0603_1608Metric, symbol Device:R_Small
- added R5: 1Meg, Resistor_SMD:R_0603_1608Metric, symbol Device:R_Small
- added R8, R9: 10, Resistor_SMD:R_0603_1608Metric, symbol Device:R_Small
- added R?: gain, Resistor_SMD:R_0603_1608Metric, symbol Device:R_Small
- added U5, U6: TSV991ILT, Package_TO_SOT_SMD:SOT-23-5_HandSoldering, symbol My_custom_lib:TSV991ILT
Connections:
- net +5V: now also C8.2, C9.2, U5.5 (V+), U6.5 (V+)
- net GND: now also C8.1, C9.1, R5.1, U5.2 (V-), U6.2 (V-)
- net at U4.1 (REFERENCE): now also Q1.1 (D), R7.1
- net at U4.2 (SENSING): now also Q1.2 (S), R8.2
- net at U4.3 (COUNTER): now also C7.1, U6.1
- new net: R10.1, U6.3 (+)
- new net: Q1.3 (G), R5.2
- new net: C?.2, R8.1, R?.2, U5.4 (-)
- new net: C7.2, R6.1, R7.2
- new net: R6.2, U6.4 (-)
- new net: R9.2, U5.3 (+)
- new net OUT3: C?.1, R?.1, U5.1
- new net REF: R10.2, R9.1
Other:
- moved on the sheet: C1, C2, C3, C4, C5, C6, R1, R2, R3, R4, U1, U2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

Commit message: u
Parts:
- removed C3, C5: 2u2, Capacitor_SMD:C_0603_1608Metric, symbol Device:C_Small
- removed C4, C6: 3n3, Capacitor_SMD:C_0603_1608Metric, symbol Device:C_Small
- removed C7, C8, C9, C?: 100n, Capacitor_SMD:C_0603_1608Metric, symbol Device:C_Small
- removed Q1: Q_PJFET_DSG, Package_TO_SOT_SMD:SOT-23, symbol Device:Q_PJFET_DSG
- removed R10, R6, R7: 10k, Resistor_SMD:R_0603_1608Metric, symbol Device:R_Small
- removed R3, R4, R5: 1Meg, Resistor_SMD:R_0603_1608Metric, symbol Device:R_Small
- removed R8, R9: 10, Resistor_SMD:R_0603_1608Metric, symbol Device:R_Small
- removed R?: gain, Resistor_SMD:R_0603_1608Metric, symbol Device:R_Small
- removed U1: USEQGCDACH4100, Z_mycustom_footprint_lib:KEMET-4-PIN-GAS-SENSOR, symbol My_custom_lib:USEQGCDACH4100
- removed U2, U3, U5, U6: TSV991ILT, Package_TO_SOT_SMD:SOT-23-5_HandSoldering, symbol My_custom_lib:TSV991ILT
- removed U4: EC4-1000-H2, symbol My_custom_lib:EC4-1000-H2
- added C? (x4): 2u2, Capacitor_SMD:C_0603_1608Metric, symbol Device:C_Small
- added FB1: FerriteBead_Small, symbol Device:FerriteBead_Small
- added J1: USB_C_Receptacle, Connector_USB:USB_C_Receptacle_HRO_TYPE-C-31-M-12, symbol Connector:USB_C_Receptacle
- added L?: L_Small, Inductor_SMD:L_0603_1608Metric, symbol Device:L_Small
- added U1: AMS1117-3.3, Package_TO_SOT_SMD:SOT-223-3_TabPin2, symbol Regulator_Linear:AMS1117-3.3
- added U2: SRV05-4, Package_TO_SOT_SMD:SOT-23-6, symbol Power_Protection:SRV05-4
- C1, C2: value 100n -> 10u; footprint Capacitor_SMD:C_0603_1608Metric -> Capacitor_SMD:C_0805_2012Metric; LCSC C14663 -> C15850
- R1, R2: value 56k -> 5k1; footprint Resistor_SMD:R_0603_1608Metric -> Resistor_SMD:R_0603_1608Metric_Pad0.98x0.95mm_HandSolder; LCSC C23206 -> C23186
Connections:
- net V-gas is gone; now on net GND: R2.2
- net V-ref is gone; now on net GND: R1.2
- net +5V: now also C?.2, C?.2, L?.2; no longer C1.2, C2.2
- net GND: now also C1.2, C2.2, C?.1, C?.1, C?.1, C?.1, J1.A1 (GND), J1.A12 (GND), J1.B1 (GND), J1.B12 (GND), U1.1 (GND), U2.2 (VN); no longer C1.1, C2.1
- net cc2: now reaches R2.1
- net cc2: now also J1.B5 (CC2)
- net cc1: now reaches R1.1
- net cc1: now also J1.A5 (CC1)
- new net: C1.1, C?.2, C?.2, FB1.1, L?.1, U1.3 (VI)
- new net +3V3: C2.1, U1.2 (VO)
- new net D+: J1.A6 (D+), J1.B6 (D+), U2.4 (IO3)
- new net D-: J1.A7 (D-), J1.B7 (D-), U2.6 (IO4)
- new net VBUS: FB1.2, J1.A4 (VBUS), J1.A9 (VBUS), J1.B4 (VBUS), J1.B9 (VBUS), U2.5 (VP)
- no-connect marks 0 -> 13
Other:
- added sheet MCU (MCU.kicad_sch)
- added sheet Measurements (Measurements.kicad_sch)
- note removed: "1.2 V, 0.1 A or 25 mW absolute max but in practice under 0.7v"

Commit message: t
Parts:
- removed C? (x2): 2u2, Capacitor_SMD:C_0603_1608Metric, symbol Device:C_Small
- added C3, C6: 10u, Capacitor_SMD:C_0805_2012Metric, symbol Device:C_Small
- added TP1, TP2: TestPoint, TestPoint:TestPoint_THTPad_2.0x2.0mm_Drill1.0mm, symbol Connector:TestPoint
- gave numbers to parts that had none: 3
Connections:
- net +3V3: now also TP1.1
- net +5V: now also C6.1, TP2.1
- net GND: now also C3.2, C6.2
- net at C1.1, C4.2, FB1.1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: now also C3.1
Other:
- moved on the sheet: C5

Commit message: o
Other:
- sheet Measurements renamed GAS_Measurements
Changed lines of the file:
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@@
     (stroke (width 0.1524) (type solid) (color 0 0 0 0))
     (fill (color 0 0 0 0.0000))
-    (property "Sheet name" "Measurements" (id 0) (at 195.58 34.8484 0)
+    (property "Sheet name" "GAS_Measurements" (id 0) (at 195.58 34.8484 0)
       (effects (font (size 1.27 1.27)) (justify left bottom))
     )

Commit message: G
Parts:
- removed TP2: TestPoint, TestPoint:TestPoint_THTPad_2.0x2.0mm_Drill1.0mm, symbol Connector:TestPoint
- added TP?: TestPoint, TestPoint:TestPoint_Pad_1.5x1.5mm, symbol Connector:TestPoint
- TP1: footprint TestPoint:TestPoint_THTPad_2.0x2.0mm_Drill1.0mm -> TestPoint:TestPoint_Pad_1.5x1.5mm
Connections:
- net +5V: now also TP?.1
Changed lines of the file:
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@@
-    (pin "1")
-  )
-  (symbol (lib_id "Connector:TestPoint") (at 154.94 55.88 0) (unit 1)
-    (in_bom no) (on_board yes)
-    (property "Reference" "TP2" (id 0) (at 154.9399 50.8 0)
-      (effects (font (size 1.27 1.27)) (justify left))
-    )
-    (property "Value" "TestPoint" (id 1) (at 157.48 53.8479 0)
-      (effects (font (size 1.27 1.27)) (justify left) hide)
-    )
-    (property "Footprint" "TestPoint:TestPoint_THTPad_2.0x2.0mm_Drill1.0mm" (id 2) (at 160.02 55.88 0)
-      (effects (font (size 1.27 1.27)) hide)
-    )
-    (property "Datasheet" "~" (id 3) (at 160.02 55.88 0)
-      (effects (font (size 1.27 1.27)) hide)
-    )
     (pin "1")
   )
@@
     )
     (property "Datasheet" "" (id 3) (at 48.26 98.425 0)
+      (effects (font (size 1.27 1.27)) hide)
+    )
+    (pin "1")
+  )
+  (symbol (lib_id "Connector:TestPoint") (at 154.94 55.88 0) (unit 1)
+    (in_bom no) (on_board yes)
+    (property "Reference" "TP?" (id 0) (at 153.67 50.165 0)
+      (effects (font (size 1.27 1.27)) (justify left))
+    )
+    (property "Value" "TestPoint" (id 1) (at 157.48 53.8479 0)
+      (effects (font (size 1.27 1.27)) (justify left) hide)
+    )
+    (property "Footprint" "TestPoint:TestPoint_Pad_1.5x1.5mm" (id 2) (at 160.02 55.88 0)
+      (effects (font (size 1.27 1.27)) hide)
+    )
+    (property "Datasheet" "~" (id 3) (at 160.02 55.88 0)
       (effects (font (size 1.27 1.27)) hide)
     )
@@
       (effects (font (size 1.27 1.27)) (justify left) hide)
     )
-    (property "Footprint" "TestPoint:TestPoint_THTPad_2.0x2.0mm_Drill1.0mm" (id 2) (at 179.705 34.925 0)
+    (property "Footprint" "TestPoint:TestPoint_Pad_1.5x1.5mm" (id 2) (at 179.705 34.925 0)
       (effects (font (size 1.27 1.27)) hide)
     )
@@
       (reference "#PWR059") (unit 1) (value "+3V3") (footprint "")
     )
+    (path "/8ec6447b-01cd-4c25-84b7-d61f3cfe2fa8/4c18df0c-39f4-43cc-b565-8284eca35f80"
+      (reference "#PWR0101") (unit 1) (value "VBUS") (footprint "")
+    )
+    (path "/8ec6447b-01cd-4c25-84b7-d61f3cfe2fa8/f2842bb5-ecf4-41a8-9d41-22c3e28e4510"
+      (reference "#PWR0102") (unit 1) (value "GND") (footprint "")
+    )
+    (path "/8ec6447b-01cd-4c25-84b7-d61f3cfe2fa8/9415a3e4-944e-478e-aece-69fc790dafd6"
+      (reference "#PWR0103") (unit 1) (value "GND") (footprint "")
+    )
     (path "/bc5bac3c-8916-4964-a51d-7cdeef038fe4"
       (reference "C1") (unit 1) (value "10u") (footprint "Capacitor_SMD:C_0805_2012Metric")
@@
       (reference "J2") (unit 1) (value "Micro_SD_Card_Det") (footprint "Connector_Card:microSD_HC_Molex_104031-0811")
     )
+    (path "/8ec6447b-01cd-4c25-84b7-d61f3cfe2fa8/4835fad9-1078-433b-85be-8d653e0113b1"
+      (reference "J3") (unit 1) (value "Conn_01x10") (footprint "")
+    )
     (path "/d3e524e5-c58d-48ef-bb76-107b5bb6bb24"
       (reference "L1") (unit 1) (value "L_Small") (footprint "Inductor_SMD:L_0603_1608Metric")
@@
       (reference "R30") (unit 1) (value "10k") (footprint "Resistor_SMD:R_0603_1608Metric_Pad0.98x0.95mm_HandSolder")
     )
-    (path "/8ec6447b-01cd-4c25-84b7-d61f3cfe2fa8/7c5eaef0-d5f2-476c-b608-4a819aab710a"
-      (reference "R31") (unit 1) (value "10") (footprint "Resistor_SMD:R_0402_1005Metric")
-    )
     (path "/4b12882e-9ea4-4ca6-b0f1-77cc2a6953ae/24f8c7d0-d0f4-437f-967e-5b6c50de8879"
       (reference "RG1") (unit 1) (value "gain") (footprint "Resistor_SMD:R_0603_1608Metric")
@@
     )
     (path "/efd7990e-4c48-4368-9b72-42872f3dbcf7"
-      (reference "TP1") (unit 1) (value "TestPoint") (footprint "TestPoint:TestPoint_THTPad_2.0x2.0mm_Drill1.0mm")
-    )
-    (path "/604d0752-765a-410c-a753-36e5ab0c5d42"
-      (reference "TP2") (unit 1) (value "TestPoint") (footprint "TestPoint:TestPoint_THTPad_2.0x2.0mm_Drill1.0mm")
-    )
-    (path "/4b12882e-9ea4-4ca6-b0f1-77cc2a6953ae/e9e6e9fe-cad4-4da8-980a-6367260b637b"
-      (reference "TP3") (unit 1) (value "TestPoint") (footprint "TestPoint:TestPoint_THTPad_2.0x2.0mm_Drill1.0mm")
-    )
-    (path "/4b12882e-9ea4-4ca6-b0f1-77cc2a6953ae/f117d029-6fd8-4a7a-b460-aca583511ff5"
-      (reference "TP4") (unit 1) (value "TestPoint") (footprint "TestPoint:TestPoint_THTPad_2.0x2.0mm_Drill1.0mm")
-    )
-    (path "/4b12882e-9ea4-4ca6-b0f1-77cc2a6953ae/e0485600-a88d-4195-b35f-8b45a1f3dfb5"
-      (reference "TP5") (unit 1) (value "TestPoint") (footprint "TestPoint:TestPoint_THTPad_2.0x2.0mm_Drill1.0mm")
-    )
-    (path "/4b12882e-9ea4-4ca6-b0f1-77cc2a6953ae/50192094-8530-40b3-bcc3-34fe8b9e24ee"
-      (reference "TP6") (unit 1) (value "TestPoint") (footprint "TestPoint:TestPoint_THTPad_2.0x2.0mm_Drill1.0mm")
-    )
-    (path "/4b12882e-9ea4-4ca6-b0f1-77cc2a6953ae/06964a60-748c-4c5e-b691-349ef2c6d67d"
-      (reference "TP7") (unit 1) (value "TestPoint") (footprint "TestPoint:TestPoint_THTPad_2.0x2.0mm_Drill1.0mm")
+      (reference "TP1") (unit 1) (value "TestPoint") (footprint "TestPoint:TestPoint_Pad_1.5x1.5mm")
+    )
+    (path "/4b12882e-9ea4-4ca6-b0f1-77cc2a6953ae/001bbaf7-594a-48a1-8501-fcb7cf01dfa9"
+      (reference "TP?") (unit 1) (value "TestPoint") (footprint "TestPoint:TestPoint_Pad_1.5x1.5mm")
+    )
+    (path "/4b12882e-9ea4-4ca6-b0f1-77cc2a6953ae/00f1ab9b-4861-417d-ba75-24a1c2f53793"
+      (reference "TP?") (unit 1) (value "TestPoint") (footprint "TestPoint:TestPoint_Pad_1.5x1.5mm")
+    )
+    (path "/4b12882e-9ea4-4ca6-b0f1-77cc2a6953ae/1cd6cdf3-d8de-45d5-ae48-857fe50290ce"
+      (reference "TP?") (unit 1) (value "TestPoint") (footprint "TestPoint:TestPoint_Pad_1.5x1.5mm")
+    )
+    (path "/4b12882e-9ea4-4ca6-b0f1-77cc2a6953ae/7890b072-4a22-47b3-b94b-4aadc7e0fa82"
+      (reference "TP?") (unit 1) (value "TestPoint") (footprint "TestPoint:TestPoint_Pad_1.5x1.5mm")
+    )
+    (path "/4b12882e-9ea4-4ca6-b0f1-77cc2a6953ae/989e6585-8eb5-4074-8154-2f24230b3ec9"
+      (reference "TP?") (unit 1) (value "TestPoint") (footprint "TestPoint:TestPoint_Pad_1.5x1.5mm")
+    )
+    (path "/baaf7cb4-5d12-4f34-a647-4aedbba17a9f"
+      (reference "TP?") (unit 1) (value "TestPoint") (footprint "TestPoint:TestPoint_Pad_1.5x1.5mm")
     )
     (path "/8946f3ac-8ac5-406e-bb7a-7095f702367f"
@@
     )
     (path "/4b12882e-9ea4-4ca6-b0f1-77cc2a6953ae/d6e5831d-ad46-4a11-9428-82f2f8142aa6"
-      (reference "U6") (unit 1) (value "EC4-1000-H2") (footprint "")
+      (reference "U6") (unit 1) (value "EC4-1000-H2") (footprint "Z_mycustom_footprint_lib:EC4-3pin")
     )
     (path "/4b12882e-9ea4-4ca6-b0f1-77cc2a6953ae/ca3b576e-eeb2-49e3-ab04-6c6e9575cc62"

Commit message: t
Parts:
- added H1, H2, H3, H4: MountingHole_Pad, MountingHole:MountingHole_3.2mm_M3_DIN965_Pad_TopBottom, symbol Mechanical:MountingHole_Pad
- gave numbers to parts that had none: 1
Connections:
- net GND: now also H1.1, H2.1, H3.1, H4.1
Changed lines of the file:
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@@
   (junction (at 127 57.15) (diameter 0) (color 0 0 0 0)
   )
+  (junction (at 295.275 57.15) (diameter 0) (color 0 0 0 0)
+  )
   (junction (at 154.94 57.15) (diameter 0) (color 0 0 0 0)
   )
@@
   )
   (junction (at 104.14 29.845) (diameter 0) (color 0 0 0 0)
+  )
+  (junction (at 295.275 52.07) (diameter 0) (color 0 0 0 0)
+  )
+  (junction (at 295.275 46.99) (diameter 0) (color 0 0 0 0)
   )
   (junction (at 175.26 29.845) (diameter 0) (color 0 0 0 0)
@@
     (stroke (width 0) (type default) (color 0 0 0 0))
   )
+  (wire (pts (xy 291.465 57.15) (xy 295.275 57.15))
+    (stroke (width 0) (type default) (color 0 0 0 0))
+  )
   (wire (pts (xy 76.2 37.465) (xy 81.28 37.465))
     (stroke (width 0) (type default) (color 0 0 0 0))
@@
     (stroke (width 0) (type default) (color 0 0 0 0))
   )
+  (wire (pts (xy 291.465 52.07) (xy 295.275 52.07))
+    (stroke (width 0) (type default) (color 0 0 0 0))
+  )
   (wire (pts (xy 164.465 29.845) (xy 172.085 29.845))
     (stroke (width 0) (type default) (color 0 0 0 0))
@@
     (stroke (width 0) (type default) (color 0 0 0 0))
   )
+  (wire (pts (xy 295.275 41.91) (xy 295.275 46.99))
+    (stroke (width 0) (type default) (color 0 0 0 0))
+  )
   (wire (pts (xy 85.09 45.085) (xy 91.44 45.085))
     (stroke (width 0) (type default) (color 0 0 0 0))
@@
     (stroke (width 0) (type default) (color 0 0 0 0))
   )
+  (wire (pts (xy 291.465 41.91) (xy 295.275 41.91))
+    (stroke (width 0) (type default) (color 0 0 0 0))
+  )
   (wire (pts (xy 154.94 57.15) (xy 160.655 57.15))
     (stroke (width 0) (type default) (color 0 0 0 0))
@@
     (stroke (width 0) (type default) (color 0 0 0 0))
   )
+  (wire (pts (xy 291.465 46.99) (xy 295.275 46.99))
+    (stroke (width 0) (type default) (color 0 0 0 0))
+  )
+  (wire (pts (xy 295.275 46.99) (xy 295.275 52.07))
+    (stroke (width 0) (type default) (color 0 0 0 0))
+  )
   (wire (pts (xy 144.145 29.845) (xy 149.225 29.845))
     (stroke (width 0) (type default) (color 0 0 0 0))
@@
     (stroke (width 0) (type default) (color 0 0 0 0))
   )
+  (wire (pts (xy 295.275 52.07) (xy 295.275 57.15))
+    (stroke (width 0) (type default) (color 0 0 0 0))
+  )
   (wire (pts (xy 66.04 47.625) (xy 66.04 50.165))
     (stroke (width 0) (type default) (color 0 0 0 0))
@@
   )
   (wire (pts (xy 135.255 60.325) (xy 135.255 57.15))
+    (stroke (width 0) (type default) (color 0 0 0 0))
+  )
+  (wire (pts (xy 295.275 57.15) (xy 295.275 59.055))
     (stroke (width 0) (type default) (color 0 0 0 0))
   )
@@
     (pin "1")
     (pin "2")
+  )
+  (symbol (lib_id "Mechanical:MountingHole_Pad") (at 288.925 46.99 90) (unit 1)
+    (in_bom no) (on_board yes)
+    (property "Reference" "H2" (id 0) (at 275.59 45.085 90))
+    (property "Value" "MountingHole_Pad" (id 1) (at 275.59 47.625 90))
+    (property "Footprint" "MountingHole:MountingHole_3.2mm_M3_DIN965_Pad_TopBottom" (id 2) (at 288.925 46.99 0)
+      (effects (font (size 1.27 1.27)) hide)
+    )
+    (property "Datasheet" "~" (id 3) (at 288.925 46.99 0)
+      (effects (font (size 1.27 1.27)) hide)
+    )
+    (pin "1")
   )
   (symbol (lib_id "Power_Protection:SRV05-4") (at 104.14 47.625 0) (mirror y) (unit 1)
@@
     (pin "1")
   )
+  (symbol (lib_id "Mechanical:MountingHole_Pad") (at 288.925 52.07 90) (unit 1)
+    (in_bom no) (on_board yes)
+    (property "Reference" "H3" (id 0) (at 275.59 50.165 90))
+    (property "Value" "MountingHole_Pad" (id 1) (at 275.59 52.705 90))
+    (property "Footprint" "MountingHole:MountingHole_3.2mm_M3_DIN965_Pad_TopBottom" (id 2) (at 288.925 52.07 0)
+      (effects (font (size 1.27 1.27)) hide)
+    )
+    (property "Datasheet" "~" (id 3) (at 288.925 52.07 0)
+      (effects (font (size 1.27 1.27)) hide)
+    )
+    (pin "1")
+  )
   (symbol (lib_id "Device:C_Small") (at 172.085 34.925 0) (unit 1)
     (in_bom yes) (on_board yes)
@@
     (pin "2")
   )
+  (symbol (lib_id "Mechanical:MountingHole_Pad") (at 288.925 57.15 90) (unit 1)
+    (in_bom no) (on_board yes)
+    (property "Reference" "H4" (id 0) (at 275.59 55.245 90))
+    (property "Value" "MountingHole_Pad" (id 1) (at 275.59 57.785 90))
+    (property "Footprint" "MountingHole:MountingHole_3.2mm_M3_DIN965_Pad_TopBottom" (id 2) (at 288.925 57.15 0)
+      (effects (font (size 1.27 1.27)) hide)
+    )
+    (property "Datasheet" "~" (id 3) (at 288.925 57.15 0)
+      (effects (font (size 1.27 1.27)) hide)
+    )
+    (pin "1")
+  )
   (symbol (lib_id "power:GND") (at 127 67.945 0) (unit 1)
     (in_bom yes) (on_board yes) (fields_autoplaced)
@@
     )
     (property "Datasheet" "" (id 3) (at 127 67.945 0)
+      (effects (font (size 1.27 1.27)) hide)
+    )
+    (pin "1")
+  )
+  (symbol (lib_id "Mechanical:MountingHole_Pad") (at 288.925 41.91 90) (unit 1)
+    (in_bom no) (on_board yes)
+    (property "Reference" "H1" (id 0) (at 275.59 40.005 90))
+    (property "Value" "MountingHole_Pad" (id 1) (at 275.59 42.545 90))
+    (property "Footprint" "MountingHole:MountingHole_3.2mm_M3_DIN965_Pad_TopBottom" (id 2) (at 288.925 41.91 0)
+      (effects (font (size 1.27 1.27)) hide)
+    )
+    (property "Datasheet" "~" (id 3) (at 288.925 41.91 0)
       (effects (font (size 1.27 1.27)) hide)
     )
@@
   (symbol (lib_id "Connector:TestPoint") (at 154.94 55.88 0) (unit 1)
     (in_bom no) (on_board yes)
-    (property "Reference" "TP?" (id 0) (at 153.67 50.165 0)
+    (property "Reference" "TP2" (id 0) (at 153.67 50.165 0)
       (effects (font (size 1.27 1.27)) (justify left))
     )
@@
     (pin "1")
   )
+  (symbol (lib_id "power:GND") (at 295.275 59.055 0) (unit 1)
+    (in_bom yes) (on_board yes) (fields_autoplaced)
+    (property "Reference" "#PWR0104" (id 0) (at 295.275 65.405 0)
+      (effects (font (size 1.27 1.27)) hide)
+    )
+    (property "Value" "GND" (id 1) (at 295.275 64.135 0)
+      (effects (font (size 1.27 1.27)) hide)
+    )
+    (property "Footprint" "" (id 2) (at 295.275 59.055 0)
+      (effects (font (size 1.27 1.27)) hide)
+    )
+    (property "Datasheet" "" (id 3) (at 295.275 59.055 0)
+      (effects (font (size 1.27 1.27)) hide)
+    )
+    (pin "1")
+  )
   (symbol (lib_id "Connector:TestPoint") (at 179.705 29.845 270) (unit 1)
     (in_bom no) (on_board yes) (fields_autoplaced)
@@
       (reference "#PWR0103") (unit 1) (value "GND") (footprint "")
     )
+    (path "/e7e4ed96-d817-4af9-b27c-cc234d6342d3"
+      (reference "#PWR0104") (unit 1) (value "GND") (footprint "")
+    )
     (path "/bc5bac3c-8916-4964-a51d-7cdeef038fe4"
       (reference "C1") (unit 1) (value "10u") (footprint "Capacitor_SMD:C_0805_2012Metric")
@@
       (reference "FB1") (unit 1) (value "FerriteBead_Small") (footprint "")
     )
+    (path "/56330439-2573-4a93-be29-14c5493ea24d"
+      (reference "H1") (unit 1) (value "MountingHole_Pad") (footprint "MountingHole:MountingHole_3.2mm_M3_DIN965_Pad_TopBottom")
+    )
+    (path "/1bc654ce-e6bc-4df7-80e8-7458e2fe27bc"
+      (reference "H2") (unit 1) (value "MountingHole_Pad") (footprint "MountingHole:MountingHole_3.2mm_M3_DIN965_Pad_TopBottom")
+    )
+    (path "/2c0799a7-0ea0-4c1e-b55e-b55474c9d385"
+      (reference "H3") (unit 1) (value "MountingHole_Pad") (footprint "MountingHole:MountingHole_3.2mm_M3_DIN965_Pad_TopBottom")
+    )
+    (path "/4427250b-97ed-4619-a23c-543eeb56cf1b"
+      (reference "H4") (unit 1) (value "MountingHole_Pad") (footprint "MountingHole:MountingHole_3.2mm_M3_DIN965_Pad_TopBottom")
+    )
     (path "/c3fdef8e-2912-4c63-81dc-d50c7f983bbe"
       (reference "J1") (unit 1) (value "USB_C_Receptacle") (footprint "Connector_USB:USB_C_Receptacle_HRO_TYPE-C-31-M-12")
@@
       (reference "TP1") (unit 1) (value "TestPoint") (footprint "TestPoint:TestPoint_Pad_1.5x1.5mm")
     )
+    (path "/baaf7cb4-5d12-4f34-a647-4aedbba17a9f"
+      (reference "TP2") (unit 1) (value "TestPoint") (footprint "TestPoint:TestPoint_Pad_1.5x1.5mm")
+    )
+    (path "/4b12882e-9ea4-4ca6-b0f1-77cc2a6953ae/989e6585-8eb5-4074-8154-2f24230b3ec9"
+      (reference "TP3") (unit 1) (value "TestPoint") (footprint "TestPoint:TestPoint_Pad_1.5x1.5mm")
+    )
     (path "/4b12882e-9ea4-4ca6-b0f1-77cc2a6953ae/001bbaf7-594a-48a1-8501-fcb7cf01dfa9"
-      (reference "TP?") (unit 1) (value "TestPoint") (footprint "TestPoint:TestPoint_Pad_1.5x1.5mm")
+      (reference "TP4") (unit 1) (value "TestPoint") (footprint "TestPoint:TestPoint_Pad_1.5x1.5mm")
     )
     (path "/4b12882e-9ea4-4ca6-b0f1-77cc2a6953ae/00f1ab9b-4861-417d-ba75-24a1c2f53793"
-      (reference "TP?") (unit 1) (value "TestPoint") (footprint "TestPoint:TestPoint_Pad_1.5x1.5mm")
+      (reference "TP5") (unit 1) (value "TestPoint") (footprint "TestPoint:TestPoint_Pad_1.5x1.5mm")
     )
     (path "/4b12882e-9ea4-4ca6-b0f1-77cc2a6953ae/1cd6cdf3-d8de-45d5-ae48-857fe50290ce"
-      (reference "TP?") (unit 1) (value "TestPoint") (footprint "TestPoint:TestPoint_Pad_1.5x1.5mm")
+      (reference "TP6") (unit 1) (value "TestPoint") (footprint "TestPoint:TestPoint_Pad_1.5x1.5mm")
     )
     (path "/4b12882e-9ea4-4ca6-b0f1-77cc2a6953ae/7890b072-4a22-47b3-b94b-4aadc7e0fa82"
-      (reference "TP?") (unit 1) (value "TestPoint") (footprint "TestPoint:TestPoint_Pad_1.5x1.5mm")
-    )
-    (path "/4b12882e-9ea4-4ca6-b0f1-77cc2a6953ae/989e6585-8eb5-4074-8154-2f24230b3ec9"
-      (reference "TP?") (unit 1) (value "TestPoint") (footprint "TestPoint:TestPoint_Pad_1.5x1.5mm")
-    )
-    (path "/baaf7cb4-5d12-4f34-a647-4aedbba17a9f"
-      (reference "TP?") (unit 1) (value "TestPoint") (footprint "TestPoint:TestPoint_Pad_1.5x1.5mm")
+      (reference "TP7") (unit 1) (value "TestPoint") (footprint "TestPoint:TestPoint_Pad_1.5x1.5mm")
     )
     (path "/8946f3ac-8ac5-406e-bb7a-7095f702367f"

Commit message: n
Parts:
- removed J1: USB_C_Receptacle, Connector_USB:USB_C_Receptacle_HRO_TYPE-C-31-M-12, symbol Connector:USB_C_Receptacle
- removed R1, R2: 5k1, Resistor_SMD:R_0603_1608Metric_Pad0.98x0.95mm_HandSolder, symbol Device:R_Small
- added J?: USB_A, SamacSys_Parts:USB1040GFLB, symbol Connector:USB_A
Connections:
- net D+: now also J?.3 (D+)
- net D-: now also J?.2 (D-)
- net GND: now also J?.4 (GND)
- net VBUS: now also J?.1 (VBUS)
- no-connect marks 13 -> 3
Other:
- moved on the sheet: C1, C2, C3, C4, C5, C6, FB1, H1, H2, H3, H4, TP1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
