File: HW/GMWPY/GMWPY.kicad_sch (KiCad schematic)
At the start: 17 parts, among them U1 AMS1117-3.3, U2 SRV05-4

Commit message: b
Parts:
- FB1: footprint (none) -> Inductor_SMD:L_0805_2012Metric
- gave numbers to parts that had none: 1
Connections:
- net D+: now also U2.1 (IO1); no longer U2.4 (IO3)
- no-connect marks 3 -> 1

Commit message: f
Parts:
- added D1, D2: RED, LED_SMD:LED_0603_1608Metric, symbol Device:LED_Small
- added R33: 1K5, Resistor_SMD:R_0603_1608Metric, symbol Device:R_Small
- added R34: 1k, Resistor_SMD:R_0603_1608Metric, symbol Device:R_Small
- added TP10, TP8, TP9: TestPoint, TestPoint:TestPoint_Pad_1.5x1.5mm, symbol Connector:TestPoint
Connections:
- net +3V3: now also R34.1
- net GND: now also D1.1 (K), D2.1 (K), TP10.1, TP8.1, TP9.1
- net VBUS: now also R33.1
- new net: D1.2 (A), R33.2
- new net: D2.2 (A), R34.2
Other:
- moved on the sheet: J1, TP1

Commit message: n
Connections:
- no-connect marks 1 -> 3
Other:
- note added: "MOUNT HOLES"
- note added: "POWER"
- moved on the sheet: C1, C2, C3, C4, C5, C6, D1, D2, FB1, J1, L1, R33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
