File: HW/GMWPY/Measurements.kicad_sch (KiCad schematic)
At the start: 35 parts, among them Q1 Q_PJFET_DSG, U10 LM4040DBZ-2.0, U3 USEQGCDACH4100, U4 TSV991ILT, U5 TSV991ILT, U6 EC4-1000-H2, U7 TSV991ILT, U8 TSV991ILT, U9 TSV991ILT

Commit message: t
Parts:
- added C7, C8: 2u2, Capacitor_SMD:C_0603_1608Metric, symbol Device:C_Small
- added RG2: gain, Resistor_SMD:R_0603_1608Metric, symbol Device:R_Small
- added TP3, TP4, TP5, TP6, TP7: TestPoint, TestPoint:TestPoint_THTPad_2.0x2.0mm_Drill1.0mm, symbol Connector:TestPoint
- renumbered C4 to C10, C5 to C11, C6 to C12, C7 to C13, C8 to C14, C9 to C15, C10 to C16, C11 to C17, C12 to C18, C13 to C19, C14 to C20, C3 to C9, R11 to R10, R12 to R11, R13 to R12, R14 to R13, R15 to R14, R16 to R15, R8 to R7, R9 to R8, R10 to R9, R7 to RG1
Connections:
- net +5V: now also C7.2, C8.2
- net GND: now also C7.1, C8.1
- net OUT1: now also TP4.1
- net OUT2: now also TP3.1
- net OUT3: now also RG2.1, TP5.1
- net REF: now also TP7.1
- net at C20.2, R13.2, R14.2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: now also TP6.1
- net at C15.2, R10.1, RG1.2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: now also RG2.2
Other:
- note added: "1.2 V, 0.1 A or 25 mW absolute max but in practice under 0.7v 25mW at 0.7V is 0.35mA FINE 25mW at 0.1V is 0.25mA FINE 25mW at 0.1A is 0.25mV unlikely"
- note added: "CH4 sensor"
- note added: "GAIN MATH: Transimpedance gain is RG in ohm H2 10-30nA/ppm so (1-3)*10^-8 0-1000ppm with 2000ppm Maximum overload Then : IF RG =10k then (10^4)*(10^-8) V/ppm => 0.1-0.3 mV/ppm with 1-3V@ 1000ppm & 2-6v@ 2000ppm"
- note added: "H2 sensor"
- note added: "Vref ~1.012V +- %"
- note added: "less then 100uA on this line"
- note removed: "1.2 V, 0.1 A or 25 mW absolute max but in practice under 0.7v"
- moved on the sheet: C10, C11, C12, C13, C14, C15, C16, C17, C18, C19, C20, C9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

Commit message: G
Parts:
- removed TP3, TP4, TP5, TP6, TP7: TestPoint, TestPoint:TestPoint_THTPad_2.0x2.0mm_Drill1.0mm, symbol Connector:TestPoint
- added TP? (x5): TestPoint, TestPoint:TestPoint_Pad_1.5x1.5mm, symbol Connector:TestPoint
- U6: footprint (none) -> Z_mycustom_footprint_lib:EC4-3pin
Connections:
- net OUT1: now also TP?.1
- net OUT2: now also TP?.1
- net OUT3: now also TP?.1
- net REF: now also TP?.1
- net H2_V+: now reaches R11.2, U7.3 (+)
- net H2_reference: now reaches Q1.1 (D), R9.1, U6.1 (REFERENCE)
- net 2V048: now reaches C20.2, R13.2, R14.2, U10.1 (K)
- net 2V048: now also TP?.1
- net 1V012: now reaches R14.1, R15.1, U9.3 (+)
- net H2_V-: now reaches C15.2, R10.1, RG1.2, RG2.2, U7.4 (-)
- net H2_sensing: now reaches Q1.2 (S), R10.2, U6.2 (SENSING)
- net H2_counter: now reaches C16.1, U6.3 (COUNTER), U8.1
- net Gas renamed CH4_Gas
- net Ref renamed CH4_Ref
- net V-gas renamed CH4_V-gas
- net V-ref renamed CH4_V-ref

Commit message: t
Parts:
- gave numbers to parts that had none: 5
Changed lines of the file:
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@@
   (symbol (lib_id "Connector:TestPoint") (at 95.25 61.595 0) (unit 1)
     (in_bom no) (on_board yes) (fields_autoplaced)
-    (property "Reference" "TP?" (id 0) (at 97.155 58.2929 0)
+    (property "Reference" "TP4" (id 0) (at 97.155 58.2929 0)
       (effects (font (size 1.27 1.27)) (justify left))
     )
@@
   (symbol (lib_id "Connector:TestPoint") (at 150.495 152.4 0) (unit 1)
     (in_bom no) (on_board yes) (fields_autoplaced)
-    (property "Reference" "TP?" (id 0) (at 153.035 149.0979 0)
+    (property "Reference" "TP5" (id 0) (at 153.035 149.0979 0)
       (effects (font (size 1.27 1.27)) (justify left))
     )
@@
   (symbol (lib_id "Connector:TestPoint") (at 48.26 206.375 0) (unit 1)
     (in_bom no) (on_board yes) (fields_autoplaced)
-    (property "Reference" "TP?" (id 0) (at 50.8 203.0729 0)
+    (property "Reference" "TP6" (id 0) (at 50.8 203.0729 0)
       (effects (font (size 1.27 1.27)) (justify left))
     )
@@
   (symbol (lib_id "Connector:TestPoint") (at 93.345 223.52 270) (unit 1)
     (in_bom no) (on_board yes) (fields_autoplaced)
-    (property "Reference" "TP?" (id 0) (at 98.425 223.5199 90)
+    (property "Reference" "TP7" (id 0) (at 98.425 223.5199 90)
       (effects (font (size 1.27 1.27)) (justify left))
     )
@@
   (symbol (lib_id "Connector:TestPoint") (at 143.51 57.15 0) (unit 1)
     (in_bom no) (on_board yes) (fields_autoplaced)
-    (property "Reference" "TP?" (id 0) (at 145.415 53.8479 0)
+    (property "Reference" "TP3" (id 0) (at 145.415 53.8479 0)
       (effects (font (size 1.27 1.27)) (justify left))
     )

Commit message: n
Parts:
- added C? (x4): 10u, Capacitor_SMD:C_0805_2012Metric, symbol Device:C_Small
- added C? (x2): 2u2, Capacitor_SMD:C_0603_1608Metric, symbol Device:C_Small
- added L?: L_Small, Inductor_SMD:L_0603_1608Metric, symbol Device:L_Small
- added U? (x2): MCP3422, symbol Analog_ADC:MCP3422
Connections:
- net GND: now also C?.1, C?.1, C?.2, C?.2, C?.2, C?.2, U?.2 (CH1-), U?.6 (Vss), U?.6 (Vss), U?.8 (CH2-), U?.8 (CH2-)
- net OUT1: now also U?.1 (CH1+)
- net OUT2: now also U?.7 (CH2+)
- net OUT3: now also U?.1 (CH1+)
- net REF: now also U?.2 (CH1-), U?.7 (CH2+)
- net 1V012 renamed 1V024
- new net +3.3VA: C?.1, C?.1, C?.1, C?.2, C?.2, L?.1, U?.3 (Vdd), U?.3 (Vdd)
- new net +3V3: C?.1, L?.2
- new net SCL: U?.5 (SCL), U?.5 (SCL)
- new net SDA: U?.4 (SDA), U?.4 (SDA)
- no-connect marks 0 -> 3
Other:
- note added: "Vref ~1.024V +- %"
- note removed: "Vref ~1.012V +- %"
- moved on the sheet: C10, C11, C12, C13, C14, C15, C16, C17, C18, C19, C20, C7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

Commit message: b
Parts:
- added C15: 2u2, Capacitor_SMD:C_0603_1608Metric, symbol Device:C_Small
- added J2: Conn_02x02_Odd_Even, Connector_PinHeader_2.54mm:PinHeader_2x02_P2.54mm_Vertical, symbol Connector_Generic:Conn_02x02_Odd_Even
- added JP1: ADR0, Jumper:SolderJumper-3_P1.3mm_Bridged12_RoundedPad1.0x1.5mm_NumberLabels, symbol Jumper:SolderJumper_3_Bridged12
- added U7: BME280, Package_LGA:Bosch_LGA-8_2.5x2.5mm_P0.65mm_ClockwisePinNumbering, symbol Sensor:BME280
- U5, U8: renamed from U?; footprint (none) -> Package_SO:SOIC-8_3.9x4.9mm_P1.27mm
- gave numbers to parts that had none: 7
- renumbered C8 to C10, C9 to C11, C10 to C14, C11 to C16, C12 to C17, C13 to C18, C14 to C19, C15 to C22, C16 to C23, C17 to C24, C18 to C25, C19 to C26, C20 to C27, C7 to C9, R3 to R1, R12 to R10, R13 to R11, R14 to R12, R15 to R13, R4 to R2, R5 to R3, R6 to R4, R7 to R5, R8 to R6, R9 to R7, R10 to R8, R11 to R9, RG2 to RG1, RG1 to RG2, U7 to U10, U8 to U11, U9 to U12, U10 to U13, U5 to U6, U6 to U9
Connections:
- net +3.3VA: now also C15.2, JP1.3 (B), U7.2 (CSB), U7.6 (VDDIO), U7.8 (VDD)
- net +3V3: now also J2.2 (Pin_2)
- net GND: now also C15.1, J2.3 (Pin_3), JP1.1 (A), U7.1 (GND), U7.7 (GND)
- net OUT1: now also U5.7 (CH2+); no longer U5.1 (CH1+)
- net OUT2: now also U5.1 (CH1+); no longer U5.7 (CH2+)
- net SCL: now also J2.1 (Pin_1), U7.4 (SCK)
- net SDA: now also J2.4 (Pin_4), U7.3 (SDI)
- new net ADRESS_BME280: JP1.2 (C), U7.5 (SDO)
Other:
- note added: "AIR MONITORING SENSORS"

Commit message: f
Parts:
- added JP2: ADR0, Jumper:SolderJumper-3_P1.3mm_Bridged12_RoundedPad1.0x1.5mm_NumberLabels, symbol Jumper:SolderJumper_3_Bridged12
- RG2: LCSC x -> C25804
Connections:
- net GND: now also JP2.3 (B)
- net REF: now also JP2.1 (A); no longer R9.1
- new net: JP2.2 (C), R9.1
Changed lines of the file:
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@@
+    (stroke (width 0) (type default) (color 0 0 0 0))
+  )
+  (wire (pts (xy 109.22 158.75) (xy 119.38 158.75))
     (stroke (width 0) (type default) (color 0 0 0 0))
   )
@@
     (stroke (width 0) (type default) (color 0 0 0 0))
   )
+  (wire (pts (xy 116.84 163.83) (xy 116.84 162.56))
+    (stroke (width 0) (type default) (color 0 0 0 0))
+  )
   (wire (pts (xy 135.89 163.83) (xy 135.89 165.1))
     (stroke (width 0) (type default) (color 0 0 0 0))
@@
     (stroke (width 0) (type default) (color 0 0 0 0))
   )
+  (wire (pts (xy 100.33 162.56) (xy 104.14 162.56))
+    (stroke (width 0) (type default) (color 0 0 0 0))
+  )
   (wire (pts (xy 316.23 95.885) (xy 316.23 97.79))
     (stroke (width 0) (type default) (color 0 0 0 0))
@@
     (stroke (width 0) (type default) (color 0 0 0 0))
   )
-  (wire (pts (xy 116.84 158.75) (xy 119.38 158.75))
-    (stroke (width 0) (type default) (color 0 0 0 0))
-  )
   (wire (pts (xy 226.06 62.23) (xy 223.52 62.23))
     (stroke (width 0) (type default) (color 0 0 0 0))
@@
   )
   (wire (pts (xy 60.96 58.42) (xy 60.96 46.99))
+    (stroke (width 0) (type default) (color 0 0 0 0))
+  )
+  (wire (pts (xy 116.84 162.56) (xy 114.3 162.56))
     (stroke (width 0) (type default) (color 0 0 0 0))
   )
@@
   )
   (text " 1.2 V, 0.1 A or 25 mW absolute max\nbut in practice under 0.7v\n25mW at 0.7V is 0.35mA  FINE\n25mW at 0.1V is 0.25mA  FINE\n25mW at 0.1A is 0.25mV  unlikely"
-    (at 73.025 175.26 0)
+    (at 58.42 179.07 0)
     (effects (font (size 1.27 1.27)) (justify left bottom))
   )
@@
     )
   )
-  (global_label "REF" (shape input) (at 116.84 158.75 180) (fields_autoplaced)
+  (global_label "REF" (shape input) (at 100.33 162.56 180) (fields_autoplaced)
     (effects (font (size 1.27 1.27)) (justify right))
-    (property "Intersheet References" "${INTERSHEET_REFS}" (id 0) (at 110.9193 158.6706 0)
+    (property "Intersheet References" "${INTERSHEET_REFS}" (id 0) (at 94.4093 162.4806 0)
       (effects (font (size 1.27 1.27)) (justify right) hide)
     )
@@
       (effects (font (size 1.27 1.27)) hide)
     )
-    (property "LCSC" "x" (id 4) (at 138.43 129.54 0)
+    (property "LCSC" "C25804" (id 4) (at 138.43 129.54 0)
       (effects (font (size 1.27 1.27)) hide)
     )
@@
     (pin "1")
   )
+  (symbol (lib_id "Jumper:SolderJumper_3_Bridged12") (at 109.22 162.56 0) (mirror x) (unit 1)
+    (in_bom no) (on_board yes)
+    (property "Reference" "JP2" (id 0) (at 109.22 167.64 0))
+    (property "Value" "ADR0" (id 1) (at 109.22 170.18 0))
+    (property "Footprint" "Jumper:SolderJumper-3_P1.3mm_Bridged12_RoundedPad1.0x1.5mm_NumberLabels" (id 2) (at 109.22 162.56 0)
+      (effects (font (size 1.27 1.27)) hide)
+    )
+    (property "Datasheet" "~" (id 3) (at 109.22 162.56 0)
+      (effects (font (size 1.27 1.27)) hide)
+    )
+    (pin "1")
+    (pin "2")
+    (pin "3")
+  )
   (symbol (lib_id "power:GND") (at 193.04 152.4 0) (unit 1)
     (in_bom yes) (on_board yes) (fields_autoplaced)
@@
     (pin "2")
   )
+  (symbol (lib_id "power:GND") (at 116.84 163.83 0) (unit 1)
+    (in_bom yes) (on_board yes) (fields_autoplaced)
+    (property "Reference" "#PWR0108" (id 0) (at 116.84 170.18 0)
+      (effects (font (size 1.27 1.27)) hide)
+    )
+    (property "Value" "GND" (id 1) (at 116.84 168.91 0)
+      (effects (font (size 1.27 1.27)) hide)
+    )
+    (property "Footprint" "" (id 2) (at 116.84 163.83 0)
+      (effects (font (size 1.27 1.27)) hide)
+    )
+    (property "Datasheet" "" (id 3) (at 116.84 163.83 0)
+      (effects (font (size 1.27 1.27)) hide)
+    )
+    (pin "1")
+  )
   (symbol (lib_id "power:GND") (at 74.93 231.14 0) (unit 1)

Commit message: f
Other:
- note added: "ADC1"
- note added: "ADC2"
Changed lines of the file:
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@@
     (effects (font (size 3 3)) (justify left bottom))
+  )
+  (text "ADC1" (at 224.79 73.66 0)
+    (effects (font (size 1.27 1.27)) (justify left bottom))
   )
   (text "less then 100uA on this line" (at 97.155 222.885 0)
@@
     (effects (font (size 5 5)) (justify left bottom))
   )
+  (text "ADC2" (at 226.06 133.35 0)
+    (effects (font (size 1.27 1.27)) (justify left bottom))
+  )
   (label "CH4_Gas" (at 60.96 63.5 0)
