File: HW/GMWPY/Measurements.kicad_sch (KiCad schematic)
At the start: 57 parts, among them J2 Conn_02x02_Odd_Even, Q1 Q_PJFET_DSG, U10 TSV991ILT, U11 TSV991ILT, U12 TSV991ILT, U13 LM4040DBZ-2.0, U3 USEQGCDACH4100, U4 TSV991ILT, U5 MCP3422, U6 TSV991ILT, U7 BME280, U8 MCP3422, U9 EC4-1000-H2

Commit message: f
Other:
- moved on the sheet: C12, C13, C7, C8, J2, L2, U5
