File: HW/GMWPY/MCU.kicad_sch (KiCad schematic)
At the start: 28 parts, among them J2 Micro_SD_Card_Det, SW1 MCU_RESET, SW2 MCU_RESET, U11 ESP32-S3-WROOM-1

Commit message: t
Parts:
- removed C17: 100n, Capacitor_SMD:C_0603_1608Metric_Pad1.08x0.95mm_HandSolder, symbol Device:C_Small
- removed C20: DNP, Capacitor_SMD:C_0603_1608Metric_Pad1.08x0.95mm_HandSolder, symbol Device:C_Small
- added C25: 10u, Capacitor_SMD:C_0805_2012Metric, symbol Device:C_Small
- C22: value 100n -> 2u2; footprint Capacitor_SMD:C_0603_1608Metric_Pad1.08x0.95mm_HandSolder -> Capacitor_SMD:C_0603_1608Metric; LCSC C14663 -> C23630
- renumbered C15 to C23, C16 to C24, C18 to C26, C19 to C27, R31 to R16, R32 to R17, R17 to R18, R18 to R19, R19 to R20, R20 to R21, R21 to R22, R22 to R23, R23 to R24, R24 to R25, R25 to R26, R26 to R27, R27 to R28, R28 to R29, R29 to R30, R30 to R31
Connections:
- net +3V3: now also C25.1
- net ESP_BOOT: now also C22.2; no longer C22.1
- net GND: now also C22.1, C25.2; no longer C22.2
Other:
- moved on the sheet: C24, R16

Commit message: G
Parts:
- removed R31: 10, Resistor_SMD:R_0402_1005Metric, symbol Device:R_Small
- added J3: Conn_01x10, symbol Connector_Generic:Conn_01x10
Connections:
- net CARD_DETECT is gone; now on net GPIO_40: J2.10 (DET_A), R30.1
- net GND: now also J3.1 (Pin_1), J3.3 (Pin_3)
- new net I2C_2_SCL: J3.5 (Pin_5)
- new net I2C_2_SDA: J3.4 (Pin_4)
- new net VBUS: J3.2 (Pin_2)
Other:
- moved on the sheet: R18, R19, R20, R21, R22, R23, R24, R25, R26, R27, R28, R29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

Commit message: n
Parts:
- added R? (x2): DNP, Resistor_SMD:R_0603_1608Metric_Pad0.98x0.95mm_HandSolder, symbol Device:R_Small
- added R? (x2): 10k, Resistor_SMD:R_0603_1608Metric_Pad0.98x0.95mm_HandSolder, symbol Device:R_Small
- J3: footprint (none) -> Connector_PinHeader_2.54mm:PinHeader_1x06_P2.54mm_Vertical; now left out of the parts list
Connections:
- net I2C_2_SCL is gone; now on net GND: J3.5 (Pin_5)
- net I2C_2_SDA is gone; now on net GPIO_5: J3.4 (Pin_4)
- net +3V3: now also J3.6 (Pin_6), R?.1, R?.1, R?.1, R?.1
- net GND: now also J3.2 (Pin_2); no longer J3.1 (Pin_1), J3.3 (Pin_3)
- net GPIO_5: now also R?.2, R?.2
- net GPIO_6: now also J3.3 (Pin_3), R?.2, R?.2
- net VBUS: now also J3.1 (Pin_1); no longer J3.2 (Pin_2)
Other:
- moved on the sheet: C21, C22, C24, C25, J3, R16, R17, SW1, SW2

Commit message: b
Parts:
- removed R27, R28, R29, R30: 10k, Resistor_SMD:R_0603_1608Metric_Pad0.98x0.95mm_HandSolder, symbol Device:R_Small
- added R21, R22, R23, R24: 10k, Resistor_SMD:R_0402_1005Metric, symbol Device:R_Small
- R20: renamed from R24; footprint Resistor_SMD:R_0603_1608Metric_Pad0.98x0.95mm_HandSolder -> Resistor_SMD:R_0402_1005Metric; LCSC C25804 -> C25744
- R25, R26: footprint Resistor_SMD:R_0603_1608Metric_Pad0.98x0.95mm_HandSolder -> Resistor_SMD:R_0402_1005Metric; LCSC C25804 -> C25744
- gave numbers to parts that had none: 4
- renumbered C21 to C28, C22 to C29, C23 to C30, C24 to C31, C25 to C32, C26 to C33, C27 to C34, J2 to J4, R16 to R14, R17 to R15, R18 to R27, R19 to R28, R20 to R29, R21 to R30, R22 to R31, R23 to R32, U11 to U14
Connections:
- net +3V3: now also R21.2, R22.2, R23.2, R24.2
- net CLK: now also R25.1
- net CMD: now also R24.1
- net DATA_1: now also R21.1; no longer R25.1
- net DATA_2: now also R22.1; no longer R26.1
- net DATA_3: now also R23.1
- net GPIO_40: now also R26.1

Commit message: f
Parts:
- added D3: RED, LED_SMD:LED_0603_1608Metric, symbol Device:LED_Small
- added R35: 1k, Resistor_SMD:R_0603_1608Metric, symbol Device:R_Small
Connections:
- net GND: now also D3.1 (K)
- net GPIO_9: now also R35.1
- new net: D3.2 (A), R35.2
Changed lines of the file:
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@@
+    (stroke (width 0) (type default) (color 0 0 0 0))
+  )
+  (wire (pts (xy 251.46 173.99) (xy 251.46 177.8))
     (stroke (width 0) (type default) (color 0 0 0 0))
   )
@@
     (stroke (width 0) (type default) (color 0 0 0 0))
   )
+  (wire (pts (xy 251.46 194.31) (xy 251.46 191.77))
+    (stroke (width 0) (type default) (color 0 0 0 0))
+  )
   (wire (pts (xy 194.31 238.76) (xy 194.31 252.73))
     (stroke (width 0) (type default) (color 0 0 0 0))
@@
   )
   (wire (pts (xy 134.62 193.04) (xy 142.24 193.04))
+    (stroke (width 0) (type default) (color 0 0 0 0))
+  )
+  (wire (pts (xy 251.46 182.88) (xy 251.46 186.69))
     (stroke (width 0) (type default) (color 0 0 0 0))
   )
@@
     (property "Intersheet References" "${INTERSHEET_REFS}" (id 0) (at 318.4012 143.4306 0)
       (effects (font (size 1.27 1.27)) (justify left) hide)
+    )
+  )
+  (global_label "GPIO_9" (shape bidirectional) (at 251.46 173.99 180) (fields_autoplaced)
+    (effects (font (size 1.27 1.27)) (justify right))
+    (property "Intersheet References" "${INTERSHEET_REFS}" (id 0) (at 242.3945 173.9106 0)
+      (effects (font (size 1.27 1.27)) (justify right) hide)
     )
   )
@@
     )
     (pin "1")
+  )
+  (symbol (lib_id "Device:LED_Small") (at 251.46 189.23 90) (unit 1)
+    (in_bom yes) (on_board yes)
+    (property "Reference" "D3" (id 0) (at 246.4435 187.96 90))
+    (property "Value" "RED" (id 1) (at 246.4435 190.5 90))
+    (property "Footprint" "LED_SMD:LED_0603_1608Metric" (id 2) (at 251.46 189.23 90)
+      (effects (font (size 1.27 1.27)) hide)
+    )
+    (property "Datasheet" "~" (id 3) (at 251.46 189.23 90)
+      (effects (font (size 1.27 1.27)) hide)
+    )
+    (property "LCSC" "C2286" (id 4) (at 251.46 189.23 0)
+      (effects (font (size 1.27 1.27)) hide)
+    )
+    (pin "1")
+    (pin "2")
   )
   (symbol (lib_id "power:+3V3") (at 307.34 120.65 0) (unit 1)
@@
     (pin "1")
   )
+  (symbol (lib_id "power:GND") (at 251.46 194.31 0) (mirror y) (unit 1)
+    (in_bom yes) (on_board yes) (fields_autoplaced)
+    (property "Reference" "#PWR0104" (id 0) (at 251.46 200.66 0)
+      (effects (font (size 1.27 1.27)) hide)
+    )
+    (property "Value" "GND" (id 1) (at 251.46 199.39 0)
+      (effects (font (size 1.27 1.27)) hide)
+    )
+    (property "Footprint" "" (id 2) (at 251.46 194.31 0)
+      (effects (font (size 1.27 1.27)) hide)
+    )
+    (property "Datasheet" "" (id 3) (at 251.46 194.31 0)
+      (effects (font (size 1.27 1.27)) hide)
+    )
+    (pin "1")
+  )
   (symbol (lib_id "power:+3V3") (at 163.83 229.87 0) (unit 1)
     (in_bom yes) (on_board yes) (fields_autoplaced)
@@
       (effects (font (size 1.27 1.27)) hide)
     )
+    (pin "1")
+    (pin "2")
+  )
+  (symbol (lib_id "Device:R_Small") (at 251.46 180.34 0) (unit 1)
+    (in_bom yes) (on_board yes)
+    (property "Reference" "R35" (id 0) (at 250.19 179.07 0)
+      (effects (font (size 1.27 1.27)) (justify right))
+    )
+    (property "Value" "1k" (id 1) (at 250.19 181.61 0)
+      (effects (font (size 1.27 1.27)) (justify right))
+    )
+    (property "Footprint" "Resistor_SMD:R_0603_1608Metric" (id 2) (at 251.46 180.34 0)
+      (effects (font (size 1.27 1.27)) hide)
+    )
+    (property "Datasheet" "~" (id 3) (at 251.46 180.34 0)
+      (effects (font (size 1.27 1.27)) hide)
+    )
+    (property "LCSC" "C21190" (id 4) (at 251.46 180.34 0)
+      (effects (font (size 1.27 1.27)) hide)
+    )

Commit message: f
Parts:
- added D4: RED, LED_SMD:LED_0603_1608Metric, symbol Device:LED_Small
- added R36, R37: 10k, Resistor_SMD:R_0603_1608Metric_Pad0.98x0.95mm_HandSolder, symbol Device:R_Small
- added R38: 1k, Resistor_SMD:R_0603_1608Metric, symbol Device:R_Small
Connections:
- net +3V3: now also R36.1, R37.1
- net GND: now also D4.1 (K)
- net GPIO_47: now also R36.2
- net GPIO_48: now also R37.2
- net GPIO_8: now also R38.1
- new net: D4.2 (A), R38.2
Other:
- moved on the sheet: C28, C29, R14, R15, SW1, SW2

Commit message: f
Other:
- note added: "MCU"
- note added: "Pull UPs"
- note added: "SD card"
- moved on the sheet: C28, C29, C30, C31, C32, C33, C34, D3, D4, J3, J4, R14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
