File: HW/GMWPY/MCU.kicad_sch (KiCad schematic)
At the start: 37 parts, among them J3 Conn_01x10, J4 Micro_SD_Card_Det, SW1 MCU_RESET, SW2 MCU_RESET, U14 ESP32-S3-WROOM-1

Commit message: b
Parts:
- added C35: 100n, Capacitor_SMD:C_0603_1608Metric_Pad1.08x0.95mm_HandSolder, symbol Device:C_Small
- added R39: 10k, Resistor_SMD:R_0603_1608Metric_Pad0.98x0.95mm_HandSolder, symbol Device:R_Small
- added SW3: MCU_RESET, SamacSys_Parts:PTS526SK15SMTR2LFS, symbol Switch:SW_SPST
Connections:
- net +3V3: now also R39.1
- net GND: now also C35.1, SW3.2 (B)
- net GPIO_16: now also C35.2, R39.2, SW3.1 (A)
Other:
- moved on the sheet: C29, R15, SW2

Commit message: n
Parts:
- added TP11, TP12, TP13: TestPoint, TestPoint:TestPoint_Pad_1.5x1.5mm, symbol Connector:TestPoint
Connections:
- net GND: now also TP13.1
- net GPIO_43: now also TP12.1
- net GPIO_44: now also TP11.1
Other:
- moved on the sheet: R16, R17, R18, R19, R36, R37
