File: HW/GMWPY/GMWPY.kicad_pcb (KiCad board)
At the start: 4 copper layers, 13 parts, among them U1 USEQGCDACH4100, U2 TSV991ILT, U3 TSV991ILT

Commit message: r
Parts:
- added C7: 100n, Capacitor_SMD:C_0603_1608Metric, F.Cu at (142.0, 101.8)
- added C8: 100n, Capacitor_SMD:C_0603_1608Metric, F.Cu at (146.9, 97.3)
- added C9: 100n, Capacitor_SMD:C_0603_1608Metric, F.Cu at (146.0, 99.9)
- added Q1: Q_PJFET_DSG, Package_TO_SOT_SMD:SOT-23, F.Cu at (138.5, 98.3)
- added R10: 10k, Resistor_SMD:R_0603_1608Metric, F.Cu at (138.0, 101.8)
- added R5: 1Meg, Resistor_SMD:R_0603_1608Metric, F.Cu at (142.9, 97.3)
- added R6: 10k, Resistor_SMD:R_0603_1608Metric, F.Cu at (138.0, 104.3)
- added R7: 10k, Resistor_SMD:R_0603_1608Metric, F.Cu at (142.0, 104.3)
- added R8: 10, Resistor_SMD:R_0603_1608Metric, F.Cu at (146.0, 104.9)
- added R9: 10, Resistor_SMD:R_0603_1608Metric, F.Cu at (146.0, 102.4)
- added U5: TSV991ILT, Package_TO_SOT_SMD:SOT-23-5_HandSoldering, F.Cu at (133.1, 98.4)
- added U6: TSV991ILT, Package_TO_SOT_SMD:SOT-23-5_HandSoldering, F.Cu at (133.1, 103.1)
Other:
- board outline added: 77.6 x 33.4 mm

Commit message: u
Parts:
- added C10: 100n, Capacitor_SMD:C_0603_1608Metric, F.Cu at (158.7, 47.2)
- added C11: 2u2, Capacitor_SMD:C_0603_1608Metric, F.Cu at (167.7, 44.7)
- added C12: 2u2, Capacitor_SMD:C_0603_1608Metric, F.Cu at (163.7, 44.7)
- added C13: 2u2, Capacitor_SMD:C_0603_1608Metric, F.Cu at (157.9, 51.3)
- added C14: 2u2, Capacitor_SMD:C_0603_1608Metric, F.Cu at (167.7, 42.2)
- added C15: 10u, Capacitor_SMD:C_0805_2012Metric, F.Cu at (98.9, 70.2)
- added C16: 10u, Capacitor_SMD:C_0805_2012Metric, F.Cu at (94.5, 70.2)
- added C17: 100n, Capacitor_SMD:C_0603_1608Metric_Pad1.08x0.95mm_HandSolder, F.Cu at (134.2, 42.2)
- added C18: 10u, Capacitor_SMD:C_0805_2012Metric, F.Cu at (115.2, 59.8)
- added C19: 100n, Capacitor_SMD:C_0603_1608Metric_Pad1.08x0.95mm_HandSolder, F.Cu at (103.3, 69.9)
- added J1: USB_C_Receptacle, Connector_USB:USB_C_Receptacle_HRO_TYPE-C-31-M-12, F.Cu at (151.9, 63.7)
- added J2: Micro_SD_Card_Det, Connector_Card:microSD_HC_Molex_104031-0811, F.Cu at (120.3, 51.2)
- added R11: 10, Resistor_SMD:R_0603_1608Metric, F.Cu at (161.9, 49.7)
- added R12: 10, Resistor_SMD:R_0603_1608Metric, F.Cu at (159.7, 42.2)
- added R13: 10k, Resistor_SMD:R_0603_1608Metric, F.Cu at (162.8, 47.2)
- added R14: 1k, Resistor_SMD:R_0603_1608Metric, F.Cu at (153.8, 51.3)
- added R15: 1k, Resistor_SMD:R_0603_1608Metric, F.Cu at (163.7, 42.2)
- added R16: 1k, Resistor_SMD:R_0603_1608Metric, F.Cu at (159.7, 44.7)
- added R17: 10, Resistor_SMD:R_0402_1005Metric, F.Cu at (129.1, 51.5)
- added R18: 10, Resistor_SMD:R_0402_1005Metric, F.Cu at (137.8, 42.0)
- added R19: 10, Resistor_SMD:R_0402_1005Metric, F.Cu at (129.1, 49.5)
- added R20: 10, Resistor_SMD:R_0402_1005Metric, F.Cu at (133.5, 47.0)
- added R21: 10, Resistor_SMD:R_0402_1005Metric, F.Cu at (111.3, 69.7)
- added R22: 10, Resistor_SMD:R_0402_1005Metric, F.Cu at (118.8, 62.3)
- added R23: 10k, Resistor_SMD:R_0603_1608Metric_Pad0.98x0.95mm_HandSolder, F.Cu at (107.7, 69.9)
- added R24: 10k, Resistor_SMD:R_0603_1608Metric_Pad0.98x0.95mm_HandSolder, F.Cu at (119.6, 59.5)
- added R25: 10k, Resistor_SMD:R_0603_1608Metric_Pad0.98x0.95mm_HandSolder, F.Cu at (129.9, 42.2)
- added R26: 10k, Resistor_SMD:R_0603_1608Metric_Pad0.98x0.95mm_HandSolder, F.Cu at (134.2, 44.7)
- added R27: 10k, Resistor_SMD:R_0603_1608Metric_Pad0.98x0.95mm_HandSolder, F.Cu at (129.9, 47.2)
- added R28: 10k, Resistor_SMD:R_0603_1608Metric_Pad0.98x0.95mm_HandSolder, F.Cu at (129.9, 44.7)
- added R29: 10k, Resistor_SMD:R_0603_1608Metric_Pad0.98x0.95mm_HandSolder, F.Cu at (115.1, 62.5)
- added R30: 10, Resistor_SMD:R_0402_1005Metric, F.Cu at (114.4, 64.8)
- added U10: LM4040DBZ-2.0, Package_TO_SOT_SMD:SOT-23, F.Cu at (154.3, 47.8)
- added U11: ESP32-S3-WROOM-1, Espressif:ESP32-S3-WROOM-1, F.Cu at (102.6, 57.6)
- added U4: TSV991ILT, Package_TO_SOT_SMD:SOT-23-5_HandSoldering, F.Cu at (154.8, 43.3)
- added U7: TSV991ILT, Package_TO_SOT_SMD:SOT-23-5_HandSoldering, F.Cu at (148.9, 47.9)
- added U8: TSV991ILT, Package_TO_SOT_SMD:SOT-23-5_HandSoldering, F.Cu at (148.9, 52.6)
- added U9: TSV991ILT, Package_TO_SOT_SMD:SOT-23-5_HandSoldering, F.Cu at (148.9, 43.3)
- C1, C2: value 100n -> 10u; footprint Capacitor_SMD:C_0603_1608Metric -> Capacitor_SMD:C_0805_2012Metric
- C4: value 3n3 -> 2u2
- C7: value 100n -> 2u2
- C8: value 100n -> 3n3
- R1, R2: value 56k -> 5k1; footprint Resistor_SMD:R_0603_1608Metric -> Resistor_SMD:R_0603_1608Metric_Pad0.98x0.95mm_HandSolder
- R3, R4: value 1Meg -> 56k
- R6: value 10k -> 1Meg
- R7: value 10k -> gain
- R8: value 10 -> 1Meg
- R9: value 10 -> 10k
- U1: value USEQGCDACH4100 -> AMS1117-3.3; footprint Z_mycustom_footprint_lib:KEMET-4-PIN-GAS-SENSOR -> Package_TO_SOT_SMD:SOT-223-3_TabPin2
- U2: value TSV991ILT -> SRV05-4; footprint Package_TO_SOT_SMD:SOT-23-5_HandSoldering -> Package_TO_SOT_SMD:SOT-23-6
- U3: value TSV991ILT -> USEQGCDACH4100; footprint Package_TO_SOT_SMD:SOT-23-5_HandSoldering -> Z_mycustom_footprint_lib:KEMET-4-PIN-GAS-SENSOR
Connections:
- C1 pad 1: GND -> +5V
- C1 pad 2: +5V -> GND
- C2 pad 1: GND -> +3V3
- C2 pad 2: +5V -> GND
- C3 pad 2: Net-(C3-Pad2) -> +5V
- C4 pad 1: /OUT2 -> GND
- C4 pad 2: /V-ref -> +5V
- C6 pad 1: /OUT1 -> /Measurements/OUT2
- C6 pad 2: /V-gas -> /Measurements/V-ref
- C7 pad 1: Net-(U4-Pad3) -> GND
- C8 pad 1: GND -> /Measurements/OUT1
- C8 pad 2: +5V -> /Measurements/V-gas
- C9 pad 1: GND -> /Measurements/OUT3
- C9 pad 2: +5V -> Net-(C9-Pad2)
- Q1 pad 1: Net-(U4-Pad1) -> Net-(Q1-Pad1)
- Q1 pad 2: Net-(U4-Pad2) -> Net-(Q1-Pad2)
- R1 pad 1: Net-(C3-Pad2) -> /cc1
- R1 pad 2: /V-ref -> GND
- R10 pad 1: Net-(R10-Pad1) -> Net-(Q1-Pad1)
- R10 pad 2: GND -> Net-(C10-Pad2)
- R2 pad 1: Net-(C5-Pad2) -> /cc2
- R2 pad 2: /V-gas -> GND
- R3 pad 1: /OUT2 -> Net-(C5-Pad2)
- R3 pad 2: /V-ref -> /Measurements/V-ref
- R4 pad 1: /OUT1 -> Net-(C7-Pad2)
- R4 pad 2: /V-gas -> /Measurements/V-gas
- R5 pad 1: GND -> /Measurements/OUT2
- R5 pad 2: Net-(Q1-Pad3) -> /Measurements/V-ref
- R6 pad 1: Net-(C7-Pad2) -> /Measurements/OUT1
- R6 pad 2: Net-(R6-Pad2) -> /Measurements/V-gas
- R7 pad 1: Net-(U4-Pad1) -> /Measurements/OUT3
- R7 pad 2: Net-(C7-Pad2) -> Net-(C9-Pad2)
- R8 pad 1: Net-(R8-Pad1) -> GND
- R8 pad 2: Net-(U4-Pad2) -> Net-(Q1-Pad3)
- R9 pad 1: GND -> Net-(C10-Pad2)
- U1 pad 2: /Ref -> +3V3
- U2 pad 1: /OUT2 -> unconnected-(U2-Pad1)
- U2 pad 3: /Ref -> unconnected-(U2-Pad3)
- U2 pad 4: /V-ref -> D+
- U2 pad 5: +5V -> VBUS
- U3 pad 1: /OUT1 -> GND
- U3 pad 2: GND -> /Measurements/Ref
- U3 pad 3: /Gas -> +5V
- U3 pad 4: /V-gas -> /Measurements/Gas
- U5 pad 1: /OUT3 -> /Measurements/OUT1
- U5 pad 3: Net-(R9-Pad2) -> /Measurements/Gas
- U5 pad 4: Net-(R8-Pad1) -> /Measurements/V-gas

Commit message: G
Parts:
- added C20: 2u2, Capacitor_SMD:C_0603_1608Metric, F.Cu at (131.8, 132.5)
- added C21: 100n, Capacitor_SMD:C_0603_1608Metric_Pad1.08x0.95mm_HandSolder, F.Cu at (111.4, 117.3)
- added C22: 2u2, Capacitor_SMD:C_0603_1608Metric, F.Cu at (133.4, 99.5)
- added C23: 10u, Capacitor_SMD:C_0805_2012Metric, F.Cu at (139.9, 89.0)
- added C24: 10u, Capacitor_SMD:C_0805_2012Metric, F.Cu at (93.9, 116.7)
- added C25: 10u, Capacitor_SMD:C_0805_2012Metric, F.Cu at (114.6, 114.6)
- added C26: 10u, Capacitor_SMD:C_0805_2012Metric, F.Cu at (98.3, 116.7)
- added C27: 100n, Capacitor_SMD:C_0603_1608Metric_Pad1.08x0.95mm_HandSolder, F.Cu at (129.3, 99.5)
- added L1: L_Small, Inductor_SMD:L_0603_1608Metric, F.Cu at (166.6, 100.0)
- added RG1: gain, Resistor_SMD:R_0603_1608Metric, F.Cu at (117.3, 150.6)
- added RG2: gain, Resistor_SMD:R_0603_1608Metric, F.Cu at (137.6, 126.3)
- added SW1: MCU_RESET, SamacSys_Parts:PTS526SK15SMTR2LFS, F.Cu at (117.9, 108.9)
- added SW2: MCU_RESET, SamacSys_Parts:PTS526SK15SMTR2LFS, F.Cu at (132.6, 91.6)
- added TP1: TestPoint, TestPoint:TestPoint_THTPad_2.0x2.0mm_Drill1.0mm, F.Cu at (178.6, 89.5)
- added TP2: TestPoint, TestPoint:TestPoint_THTPad_2.0x2.0mm_Drill1.0mm, F.Cu at (174.2, 92.5)
- added TP3: TestPoint, TestPoint:TestPoint_THTPad_2.0x2.0mm_Drill1.0mm, F.Cu at (116.8, 144.8)
- added TP4: TestPoint, TestPoint:TestPoint_THTPad_2.0x2.0mm_Drill1.0mm, F.Cu at (131.8, 129.2)
- added TP5: TestPoint, TestPoint:TestPoint_THTPad_2.0x2.0mm_Drill1.0mm, F.Cu at (133.6, 124.5)
- added TP6: TestPoint, TestPoint:TestPoint_THTPad_2.0x2.0mm_Drill1.0mm, F.Cu at (127.8, 129.2)
- added TP7: TestPoint, TestPoint:TestPoint_THTPad_2.0x2.0mm_Drill1.0mm, F.Cu at (110.2, 147.7)
- C10, C9: value 100n -> 2u2
- C12, C14: value 2u2 -> 3n3
- C15, C16: value 10u -> 100n; footprint Capacitor_SMD:C_0805_2012Metric -> Capacitor_SMD:C_0603_1608Metric
- C17, C19: value 100n -> 2u2; footprint Capacitor_SMD:C_0603_1608Metric_Pad1.08x0.95mm_HandSolder -> Capacitor_SMD:C_0603_1608Metric
- C18: value 10u -> 2u2; footprint Capacitor_SMD:C_0805_2012Metric -> Capacitor_SMD:C_0603_1608Metric
- C3: value 2u2 -> 10u; footprint Capacitor_SMD:C_0603_1608Metric -> Capacitor_SMD:C_0805_2012Metric
- C6: value 3n3 -> 10u; footprint Capacitor_SMD:C_0603_1608Metric -> Capacitor_SMD:C_0805_2012Metric
- C8: value 3n3 -> 2u2
- R10: value 10k -> 10
- R12: value 10 -> 10k
- R13: value 10k -> 1k
- R16: value 1k -> 10k; footprint Resistor_SMD:R_0603_1608Metric -> Resistor_SMD:R_0603_1608Metric_Pad0.98x0.95mm_HandSolder
- R17, R30: value 10 -> 10k; footprint Resistor_SMD:R_0402_1005Metric -> Resistor_SMD:R_0603_1608Metric_Pad0.98x0.95mm_HandSolder
- R23: value 10k -> 10; footprint Resistor_SMD:R_0603_1608Metric_Pad0.98x0.95mm_HandSolder -> Resistor_SMD:R_0402_1005Metric
- R7: value gain -> 1Meg
- R8: value 1Meg -> 10k
- U3: moved to B.Cu
- U6: value TSV991ILT -> EC4-1000-H2; footprint Package_TO_SOT_SMD:SOT-23-5_HandSoldering -> Z_mycustom_footprint_lib:EC4-3pin; moved to B.Cu
- moved U9 118.0 mm to (94.5, 148.0)
- moved C12 112.4 mm to (122.2, 149.2)
- moved C11 111.7 mm to (122.2, 146.7)
- moved U7 111.2 mm to (100.3, 148.0)
- moved C13 109.2 mm to (113.3, 151.0)
- moved C14 106.9 mm to (122.6, 139.2)
- moved U4 104.0 mm to (117.7, 140.4)
- moved C10 101.1 mm to (122.6, 141.7)
- moved R12 98.2 mm to (127.5, 135.0)
- moved R15 98.2 mm to (131.5, 135.0)
- moved U10 93.3 mm to (123.0, 135.7)
- moved R16 91.6 mm to (102.7, 116.4)
- moved C18 88.3 mm to (114.2, 148.1)
- moved R13 88.3 mm to (135.8, 131.3)
- moved C17 86.8 mm to (139.8, 128.8)
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Connections:
- net /Measurements/Gas renamed /GAS_Measurements/CH4_Gas
- net /Measurements/Ref renamed /GAS_Measurements/CH4_Ref
- C1 pad 1: +5V -> Net-(C1-Pad1)
- C10 pad 1: Net-(C10-Pad1) -> GND
- C10 pad 2: Net-(C10-Pad2) -> +5V
- C11 pad 2: +5V -> Net-(C11-Pad2)
- C12 pad 1: GND -> /GAS_Measurements/OUT2
- C12 pad 2: +5V -> /GAS_Measurements/CH4_V-ref
- C13 pad 2: +5V -> Net-(C13-Pad2)
- C14 pad 1: GND -> /GAS_Measurements/OUT1
- C14 pad 2: Net-(C14-Pad2) -> /GAS_Measurements/CH4_V-gas
- C15 pad 1: +3V3 -> /GAS_Measurements/OUT3
- C15 pad 2: GND -> /GAS_Measurements/H2_V-
- C16 pad 1: +3V3 -> /GAS_Measurements/H2_counter
- C16 pad 2: GND -> Net-(C16-Pad2)
- C17 pad 1: +3V3 -> GND
- C17 pad 2: GND -> +5V
- C18 pad 1: +3V3 -> GND
- C18 pad 2: GND -> +5V
- C19 pad 1: +3V3 -> GND
- C19 pad 2: GND -> +5V
- C3 pad 1: GND -> Net-(C1-Pad1)
- C3 pad 2: +5V -> GND
- C4 pad 2: +5V -> Net-(C1-Pad1)
- C5 pad 2: Net-(C5-Pad2) -> +5V
- C6 pad 1: /Measurements/OUT2 -> +5V
- C6 pad 2: /Measurements/V-ref -> GND
- C7 pad 2: Net-(C7-Pad2) -> +5V
- C8 pad 1: /Measurements/OUT1 -> GND
- C8 pad 2: /Measurements/V-gas -> +5V
- C9 pad 1: /Measurements/OUT3 -> GND
- C9 pad 2: Net-(C9-Pad2) -> +5V
- J2 pad 10: /MCU/CARD_DETECT -> GPIO_40
- Q1 pad 1: Net-(Q1-Pad1) -> /GAS_Measurements/H2_reference
- Q1 pad 2: Net-(Q1-Pad2) -> /GAS_Measurements/H2_sensing
- R10 pad 1: Net-(Q1-Pad1) -> /GAS_Measurements/H2_V-
- R10 pad 2: Net-(C10-Pad2) -> /GAS_Measurements/H2_sensing
- R11 pad 1: Net-(C9-Pad2) -> REF
- R11 pad 2: Net-(Q1-Pad2) -> /GAS_Measurements/H2_V+
- R12 pad 1: REF -> Net-(R12-Pad1)
- R12 pad 2: Net-(R12-Pad2) -> REF
- R13 pad 1: Net-(R13-Pad1) -> +5V
- R13 pad 2: REF -> 2V048
- R14 pad 1: +5V -> /GAS_Measurements/1V012
- R14 pad 2: Net-(C14-Pad2) -> 2V048
- R15 pad 1: Net-(R15-Pad1) -> /GAS_Measurements/1V012
- R15 pad 2: Net-(C14-Pad2) -> GND
- R16 pad 1: Net-(R15-Pad1) -> +3V3
- R16 pad 2: GND -> /MCU/ESP_EN
- R17 pad 1: /MCU/DATA_0 -> /MCU/ESP_BOOT
- R17 pad 2: GPIO_42 -> +3V3
- R18 pad 1: /MCU/DATA_1 -> /MCU/DATA_0
- R18 pad 2: GPIO_41 -> GPIO_42
- R19 pad 1: /MCU/DATA_2 -> /MCU/DATA_1
- R19 pad 2: GPIO_1 -> GPIO_41
- R20 pad 1: /MCU/DATA_3 -> /MCU/DATA_2
- R20 pad 2: GPIO_2 -> GPIO_1
- R21 pad 1: /MCU/CMD -> /MCU/DATA_3
- R21 pad 2: GPIO_43 -> GPIO_2
- R22 pad 1: /MCU/CLK -> /MCU/CMD
- R22 pad 2: GPIO_44 -> GPIO_43
- R23 pad 1: /MCU/DATA_0 -> /MCU/CLK
- R23 pad 2: +3V3 -> GPIO_44
- R24 pad 1: /MCU/DATA_1 -> /MCU/DATA_0
- R25 pad 1: /MCU/DATA_2 -> /MCU/DATA_1
- R26 pad 1: /MCU/DATA_3 -> /MCU/DATA_2
- R27 pad 1: /MCU/CMD -> /MCU/DATA_3
- R28 pad 1: /MCU/CLK -> /MCU/CMD
- R29 pad 1: /MCU/CARD_DETECT -> /MCU/CLK
- R3 pad 1: Net-(C5-Pad2) -> Net-(C11-Pad2)
- R3 pad 2: /Measurements/V-ref -> /GAS_Measurements/CH4_V-ref
- R30 pad 1: /MCU/CARD_DETECT -> GPIO_40
- R30 pad 2: GPIO_40 -> +3V3
- R4 pad 1: Net-(C7-Pad2) -> Net-(C13-Pad2)
- R4 pad 2: /Measurements/V-gas -> /GAS_Measurements/CH4_V-gas
- R5 pad 1: /Measurements/OUT2 -> /GAS_Measurements/OUT2
- R5 pad 2: /Measurements/V-ref -> /GAS_Measurements/CH4_V-ref
- R6 pad 1: /Measurements/OUT1 -> /GAS_Measurements/OUT1
- R6 pad 2: /Measurements/V-gas -> /GAS_Measurements/CH4_V-gas
- R7 pad 1: /Measurements/OUT3 -> GND
- R7 pad 2: Net-(C9-Pad2) -> Net-(Q1-Pad3)
- R8 pad 1: GND -> Net-(C16-Pad2)
- R8 pad 2: Net-(Q1-Pad3) -> Net-(R8-Pad2)
- R9 pad 1: Net-(C10-Pad2) -> /GAS_Measurements/H2_reference
- R9 pad 2: Net-(R9-Pad2) -> Net-(C16-Pad2)
- U1 pad 3: +5V -> Net-(C1-Pad1)
- U10 pad 1: Net-(C14-Pad2) -> 2V048
- U4 pad 1: /Measurements/OUT2 -> /GAS_Measurements/OUT2
- U4 pad 4: /Measurements/V-ref -> /GAS_Measurements/CH4_V-ref
- U5 pad 1: /Measurements/OUT1 -> /GAS_Measurements/OUT1
- U5 pad 4: /Measurements/V-gas -> /GAS_Measurements/CH4_V-gas
- U6 pad 1: Net-(U4-Pad3) -> /GAS_Measurements/H2_reference
- U6 pad 2: GND -> /GAS_Measurements/H2_sensing
- U6 pad 3: Net-(R10-Pad1) -> /GAS_Measurements/H2_counter
- U7 pad 1: /Measurements/OUT3 -> /GAS_Measurements/OUT3
- U7 pad 3: Net-(R12-Pad2) -> /GAS_Measurements/H2_V+
- U7 pad 4: Net-(C9-Pad2) -> /GAS_Measurements/H2_V-
- U8 pad 1: Net-(C10-Pad1) -> /GAS_Measurements/H2_counter
- U8 pad 3: Net-(R13-Pad1) -> Net-(R12-Pad1)
- U8 pad 4: Net-(R9-Pad2) -> Net-(R8-Pad2)
- U9 pad 3: Net-(R15-Pad1) -> /GAS_Measurements/1V012
Other:
- board size 77.6 x 33.4 mm -> 114.1 x 79 mm

Commit message: t
Parts:
- added H1: MountingHole_Pad, MountingHole:MountingHole_3.2mm_M3_DIN965_Pad_TopBottom, F.Cu at (156.6, 150.4)
- added H2: MountingHole_Pad, MountingHole:MountingHole_3.2mm_M3_DIN965_Pad_TopBottom, F.Cu at (149.4, 143.2)
- added H3: MountingHole_Pad, MountingHole:MountingHole_3.2mm_M3_DIN965_Pad_TopBottom, F.Cu at (149.4, 150.4)
- added H4: MountingHole_Pad, MountingHole:MountingHole_3.2mm_M3_DIN965_Pad_TopBottom, F.Cu at (156.6, 143.2)
- TP1, TP2, TP3, TP4, TP5, TP6, TP7: footprint TestPoint:TestPoint_THTPad_2.0x2.0mm_Drill1.0mm -> TestPoint:TestPoint_Pad_1.5x1.5mm
- moved TP1 79.7 mm to (128.0, 151.1), turned to 180 degrees
- moved C1 75.4 mm to (132.3, 151.6), turned to 180 degrees
- moved TP2 69.4 mm to (132.5, 148.1), turned to 180 degrees
- moved U1 63.7 mm to (139.4, 149.0), turned to 180 degrees
- moved C4 61.1 mm to (133.6, 143.6), turned to 180 degrees
- moved R2 56.1 mm to (137.7, 143.6), turned to 180 degrees
- moved C2 51.2 mm to (142.1, 143.3), turned to 180 degrees
- moved L1 48.4 mm to (140.1, 140.6), turned to 180 degrees
- moved R1 22.3 mm to (146.3, 115.4)
- moved C5 22.3 mm to (146.1, 117.9)
- moved C6 22.3 mm to (141.9, 114.8)
- moved U2 22.3 mm to (137.1, 115.6)
- moved C3 22.3 mm to (141.9, 117.8)
- moved J1 22.3 mm to (140.3, 108.7)
Other:
- board size 114.1 x 79 mm -> 77.4 x 77.2 mm

Commit message: b
Parts:
- added C28: 100n, Capacitor_SMD:C_0603_1608Metric_Pad1.08x0.95mm_HandSolder, F.Cu at (72.3, 93.9)
- added C29: 2u2, Capacitor_SMD:C_0603_1608Metric, F.Cu at (78.7, 93.9)
- added C30: 10u, Capacitor_SMD:C_0805_2012Metric, B.Cu at (68.5, 59.8)
- added C31: 10u, Capacitor_SMD:C_0805_2012Metric, F.Cu at (64.4, 59.8)
- added C32: 10u, Capacitor_SMD:C_0805_2012Metric, F.Cu at (66.4, 59.8)
- added C33: 10u, Capacitor_SMD:C_0805_2012Metric, F.Cu at (92.6, 58.1)
- added C34: 100n, Capacitor_SMD:C_0603_1608Metric_Pad1.08x0.95mm_HandSolder, B.Cu at (101.7, 58.8)
- added FB1: FerriteBead_Small, Inductor_SMD:L_0805_2012Metric, F.Cu at (58.0, 87.0)
- added J3: Conn_01x10, Connector_PinHeader_2.54mm:PinHeader_1x06_P2.54mm_Vertical, F.Cu at (91.4, 73.5)
- added J4: Micro_SD_Card_Det, Connector_Card:microSD_HC_Molex_104031-0811, F.Cu at (100.4, 64.3)
- added JP1: ADR0, Jumper:SolderJumper-3_P1.3mm_Bridged12_RoundedPad1.0x1.5mm_NumberLabels, B.Cu at (109.3, 77.7)
- added L2: L_Small, Inductor_SMD:L_0603_1608Metric, F.Cu at (78.2, 98.0)
- added R31: 10, Resistor_SMD:R_0402_1005Metric, F.Cu at (88.7, 62.8)
- added R32: 10, Resistor_SMD:R_0402_1005Metric, F.Cu at (88.7, 64.1)
- added U12: TSV991ILT, Package_TO_SOT_SMD:SOT-23-5_HandSoldering, F.Cu at (121.8, 88.1)
- added U13: LM4040DBZ-2.0, Package_TO_SOT_SMD:SOT-23, F.Cu at (115.0, 86.7)
- added U14: ESP32-S3-WROOM-1, Espressif:ESP32-S3-WROOM-1, F.Cu at (77.3, 67.3)
- C12: value 3n3 -> 10u; footprint Capacitor_SMD:C_0603_1608Metric -> Capacitor_SMD:C_0805_2012Metric
- C14: value 3n3 -> 2u2
- C15, C16: value 100n -> 2u2
- C17, C19: value 2u2 -> 3n3
- C20, C7, C8: value 2u2 -> 10u; footprint Capacitor_SMD:C_0603_1608Metric -> Capacitor_SMD:C_0805_2012Metric
- C21, C27: value 100n -> 2u2; footprint Capacitor_SMD:C_0603_1608Metric_Pad1.08x0.95mm_HandSolder -> Capacitor_SMD:C_0603_1608Metric
- C22: value 2u2 -> 100n
- C23: value 10u -> 100n; footprint Capacitor_SMD:C_0805_2012Metric -> Capacitor_SMD:C_0603_1608Metric
- C24, C25, C26: value 10u -> 2u2; footprint Capacitor_SMD:C_0805_2012Metric -> Capacitor_SMD:C_0603_1608Metric
- J1: value USB_C_Receptacle -> USB_A; footprint Connector_USB:USB_C_Receptacle_HRO_TYPE-C-31-M-12 -> SamacSys_Parts:USB1040GFLB
- J2: value Micro_SD_Card_Det -> Conn_02x02_Odd_Even; footprint Connector_Card:microSD_HC_Molex_104031-0811 -> Connector_PinHeader_2.54mm:PinHeader_2x02_P2.54mm_Vertical; moved to B.Cu
- R1, R2: value 5k1 -> 56k; footprint Resistor_SMD:R_0603_1608Metric_Pad0.98x0.95mm_HandSolder -> Resistor_SMD:R_0603_1608Metric
- R10, R20, R21, R22, R23: value 10 -> 10k
- R11: value 10 -> 1k
- R12: value 10k -> 1k
- R14, R15: value 1k -> 10k; footprint Resistor_SMD:R_0603_1608Metric -> Resistor_SMD:R_0603_1608Metric_Pad0.98x0.95mm_HandSolder
- R16: value 10k -> DNP
- R18: value 10 -> 10k; footprint Resistor_SMD:R_0402_1005Metric -> Resistor_SMD:R_0603_1608Metric_Pad0.98x0.95mm_HandSolder
- R19: value 10 -> DNP; footprint Resistor_SMD:R_0402_1005Metric -> Resistor_SMD:R_0603_1608Metric_Pad0.98x0.95mm_HandSolder
- R24, R25, R26: footprint Resistor_SMD:R_0603_1608Metric_Pad0.98x0.95mm_HandSolder -> Resistor_SMD:R_0402_1005Metric
- R27, R28, R29, R30: value 10k -> 10; footprint Resistor_SMD:R_0603_1608Metric_Pad0.98x0.95mm_HandSolder -> Resistor_SMD:R_0402_1005Metric
- R3, R4: value 56k -> 1Meg
- R6, R7: value 1Meg -> 10k
- R8, R9: value 10k -> 10
- U10: value LM4040DBZ-2.0 -> TSV991ILT; footprint Package_TO_SOT_SMD:SOT-23 -> Package_TO_SOT_SMD:SOT-23-5_HandSoldering
- U11: value ESP32-S3-WROOM-1 -> TSV991ILT; footprint Espressif:ESP32-S3-WROOM-1 -> Package_TO_SOT_SMD:SOT-23-5_HandSoldering
- U5, U8: value TSV991ILT -> MCP3422; footprint Package_TO_SOT_SMD:SOT-23-5_HandSoldering -> Package_SO:SOIC-8_3.9x4.9mm_P1.27mm
- U6: value EC4-1000-H2 -> TSV991ILT; footprint Z_mycustom_footprint_lib:EC4-3pin -> Package_TO_SOT_SMD:SOT-23-5_HandSoldering; moved to F.Cu
- U7: value TSV991ILT -> BME280; footprint Package_TO_SOT_SMD:SOT-23-5_HandSoldering -> Package_LGA:Bosch_LGA-8_2.5x2.5mm_P0.65mm_ClockwisePinNumbering; moved to B.Cu
- U9: value TSV991ILT -> EC4-1000-H2; footprint Package_TO_SOT_SMD:SOT-23-5_HandSoldering -> Z_mycustom_footprint_lib:EC4-3pin; moved to B.Cu
- moved H1 140.8 mm to (54.0, 54.0)
- moved H4 109.1 mm to (53.9, 106.3)
- moved C1 97.0 mm to (58.2, 89.0)
- moved C2 96.3 mm to (62.6, 89.0), turned to 0 degrees
- moved U1 95.0 mm to (61.5, 94.6), turned to -90 degrees
- moved H2 90.8 mm to (130.2, 54.5)
- moved J1 88.3 mm to (60.3, 71.3), turned to -90 degrees
- moved U2 83.2 mm to (64.5, 74.8), turned to 90 degrees
- moved R6 82.6 mm to (121.2, 72.4), turned to -90 degrees
- moved TP1 82.3 mm to (66.8, 96.2)
- moved R19 78.9 mm to (65.4, 64.2)
- moved U9 78.1 mm to (122.8, 75.2), turned to -45 degrees
- moved RG1 76.8 mm to (115.9, 73.8)
- moved Q1 76.2 mm to (129.4, 75.5), turned to 180 degrees
- moved R8 75.9 mm to (118.2, 76.0), turned to 90 degrees
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Connections:
- C11 pad 2: Net-(C11-Pad2) -> +5V
- C12 pad 1: /GAS_Measurements/OUT2 -> +3.3VA
- C12 pad 2: /GAS_Measurements/CH4_V-ref -> GND
- C13 pad 2: Net-(C13-Pad2) -> +3.3VA
- C14 pad 1: /GAS_Measurements/OUT1 -> GND
- C14 pad 2: /GAS_Measurements/CH4_V-gas -> +5V
- C15 pad 1: /GAS_Measurements/OUT3 -> GND
- C15 pad 2: /GAS_Measurements/H2_V- -> +3.3VA
- C16 pad 1: /GAS_Measurements/H2_counter -> GND
- C17 pad 1: GND -> /GAS_Measurements/OUT2
- C17 pad 2: +5V -> /GAS_Measurements/CH4_V-ref
- C18 pad 2: +5V -> Net-(C18-Pad2)
- C19 pad 1: GND -> /GAS_Measurements/OUT1
- C19 pad 2: +5V -> /GAS_Measurements/CH4_V-gas
- C20 pad 1: GND -> +3.3VA
- C20 pad 2: 2V048 -> GND
- C21 pad 2: /MCU/ESP_EN -> +3.3VA
- C22 pad 1: GND -> /GAS_Measurements/OUT3
- C22 pad 2: /MCU/ESP_BOOT -> /GAS_Measurements/H2_V-
- C23 pad 1: +3V3 -> /GAS_Measurements/H2_counter
- C23 pad 2: GND -> Net-(C23-Pad2)
- C24 pad 1: +3V3 -> GND
- C24 pad 2: GND -> +5V
- C25 pad 1: +3V3 -> GND
- C25 pad 2: GND -> +5V
- C26 pad 1: +3V3 -> GND
- C26 pad 2: GND -> +5V
- C27 pad 1: +3V3 -> GND
- C27 pad 2: GND -> 2V048
- C7 pad 1: GND -> +3.3VA
- C7 pad 2: +5V -> GND
- C8 pad 1: GND -> +3V3
- C8 pad 2: +5V -> GND
- J2 pad 1: /MCU/DATA_2 -> GPIO_5
- J2 pad 2: /MCU/DATA_3 -> +3V3
- J2 pad 3: /MCU/CMD -> GND
- J2 pad 4: +3V3 -> GPIO_6
- R1 pad 1: /cc1 -> Net-(C16-Pad2)
- R1 pad 2: GND -> /GAS_Measurements/CH4_V-ref
- R10 pad 1: /GAS_Measurements/H2_V- -> Net-(R10-Pad1)
- R10 pad 2: /GAS_Measurements/H2_sensing -> REF
- R11 pad 1: REF -> +5V
- R11 pad 2: /GAS_Measurements/H2_V+ -> 2V048
- R12 pad 1: Net-(R12-Pad1) -> /GAS_Measurements/1V024
- R12 pad 2: REF -> 2V048
- R13 pad 1: +5V -> /GAS_Measurements/1V024
- R13 pad 2: 2V048 -> GND
- R14 pad 1: /GAS_Measurements/1V012 -> +3V3
- R14 pad 2: 2V048 -> /MCU/ESP_EN
- R15 pad 1: /GAS_Measurements/1V012 -> /MCU/ESP_BOOT
- R15 pad 2: GND -> +3V3
- R16 pad 2: /MCU/ESP_EN -> GPIO_6
- R17 pad 1: /MCU/ESP_BOOT -> +3V3
- R17 pad 2: +3V3 -> GPIO_6
- R18 pad 1: /MCU/DATA_0 -> +3V3
- R18 pad 2: GPIO_42 -> GPIO_5
- R19 pad 1: /MCU/DATA_1 -> +3V3
- R19 pad 2: GPIO_41 -> GPIO_5
- R2 pad 1: /cc2 -> Net-(C18-Pad2)
- R2 pad 2: GND -> /GAS_Measurements/CH4_V-gas
- R20 pad 1: /MCU/DATA_2 -> /MCU/DATA_0
- R20 pad 2: GPIO_1 -> +3V3
- R21 pad 1: /MCU/DATA_3 -> /MCU/DATA_1
- R21 pad 2: GPIO_2 -> +3V3
- R22 pad 1: /MCU/CMD -> /MCU/DATA_2
- R22 pad 2: GPIO_43 -> +3V3
- R23 pad 1: /MCU/CLK -> /MCU/DATA_3
- R23 pad 2: GPIO_44 -> +3V3
- R24 pad 1: /MCU/DATA_0 -> /MCU/CMD
- R25 pad 1: /MCU/DATA_1 -> /MCU/CLK
- R26 pad 1: /MCU/DATA_2 -> GPIO_40
- R27 pad 1: /MCU/DATA_3 -> /MCU/DATA_0
- R27 pad 2: +3V3 -> GPIO_42
- R28 pad 1: /MCU/CMD -> /MCU/DATA_1
- R28 pad 2: +3V3 -> GPIO_41
- R29 pad 1: /MCU/CLK -> /MCU/DATA_2
- R29 pad 2: +3V3 -> GPIO_1
- R3 pad 1: Net-(C11-Pad2) -> /GAS_Measurements/OUT2
- R30 pad 1: GPIO_40 -> /MCU/DATA_3
- R30 pad 2: +3V3 -> GPIO_2
- R4 pad 1: Net-(C13-Pad2) -> /GAS_Measurements/OUT1
- R5 pad 1: /GAS_Measurements/OUT2 -> GND
- R5 pad 2: /GAS_Measurements/CH4_V-ref -> Net-(Q1-Pad3)
- R6 pad 1: /GAS_Measurements/OUT1 -> Net-(C23-Pad2)
- R6 pad 2: /GAS_Measurements/CH4_V-gas -> Net-(R6-Pad2)
- R7 pad 1: GND -> /GAS_Measurements/H2_reference
- R7 pad 2: Net-(Q1-Pad3) -> Net-(C23-Pad2)
- R8 pad 1: Net-(C16-Pad2) -> /GAS_Measurements/H2_V-
- R8 pad 2: Net-(R8-Pad2) -> /GAS_Measurements/H2_sensing
- R9 pad 1: /GAS_Measurements/H2_reference -> REF
- R9 pad 2: Net-(C16-Pad2) -> /GAS_Measurements/H2_V+
- U10 pad 1: 2V048 -> /GAS_Measurements/OUT3
- U10 pad 3: (no net) -> /GAS_Measurements/H2_V+
- U11 pad 1: GND -> /GAS_Measurements/H2_counter
- U11 pad 2: +3V3 -> GND
- U11 pad 3: /MCU/ESP_EN -> Net-(R10-Pad1)
- U11 pad 4: GPIO_4 -> Net-(R6-Pad2)
- U11 pad 5: GPIO_5 -> +5V
- U2 pad 1: unconnected-(U2-Pad1) -> D+
- U2 pad 4: D+ -> unconnected-(U2-Pad4)
- U5 pad 1: /GAS_Measurements/OUT1 -> /GAS_Measurements/OUT2
- U5 pad 3: /GAS_Measurements/CH4_Gas -> +3.3VA
- U5 pad 4: /GAS_Measurements/CH4_V-gas -> GPIO_6
- U5 pad 5: +5V -> GPIO_5
- U6 pad 1: /GAS_Measurements/H2_reference -> /GAS_Measurements/OUT1
- U6 pad 2: /GAS_Measurements/H2_sensing -> GND
- U6 pad 3: /GAS_Measurements/H2_counter -> /GAS_Measurements/CH4_Gas
- U7 pad 1: /GAS_Measurements/OUT3 -> GND
- U7 pad 2: GND -> +3.3VA
- U7 pad 3: /GAS_Measurements/H2_V+ -> GPIO_6
- U7 pad 4: /GAS_Measurements/H2_V- -> GPIO_5
- U7 pad 5: +5V -> /GAS_Measurements/ADRESS_BME280
- U8 pad 1: /GAS_Measurements/H2_counter -> /GAS_Measurements/OUT3
- U8 pad 2: GND -> REF
- U8 pad 3: Net-(R12-Pad1) -> +3.3VA
- U8 pad 4: Net-(R8-Pad2) -> GPIO_6
- U8 pad 5: +5V -> GPIO_5
- U9 pad 1: REF -> /GAS_Measurements/H2_reference
- U9 pad 2: GND -> /GAS_Measurements/H2_sensing
- U9 pad 3: /GAS_Measurements/1V012 -> /GAS_Measurements/H2_counter
Routing:
- net +3V3: track 0.00 -> 169.0 mm, vias 0 -> 5
- net GND: track 0.00 -> 95.9 mm, vias 0 -> 49
- net GPIO_6: track 0.00 -> 81.5 mm, vias 0 -> 4
- net GPIO_5: track 0.00 -> 77.1 mm, vias 0 -> 4
- net +5V: track 0.00 -> 38.6 mm
- net /MCU/ESP_EN: track 0.00 -> 37.7 mm, vias 0 -> 2
- net REF: track 0.00 -> 35.0 mm
- net /GAS_Measurements/H2_sensing: track 0.00 -> 25.8 mm
- net VBUS: track 0.00 -> 25.5 mm
- net /MCU/DATA_1: track 0.00 -> 23.8 mm, vias 0 -> 2
- net /MCU/ESP_BOOT: track 0.00 -> 23.3 mm, vias 0 -> 2
- net +3.3VA: track 0.00 -> 21.8 mm, vias 0 -> 2
- net /MCU/DATA_0: track 0.00 -> 21.8 mm, vias 0 -> 2
- net /GAS_Measurements/OUT1: track 0.00 -> 17.8 mm
- net /MCU/CLK: track 0.00 -> 17.7 mm, vias 0 -> 2
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- added copper zone on B.Cu, net +3V3
- added copper zone on F.Cu, net +3V3
- added copper zone on F.Cu, net GND
- added copper zone on In1.Cu, net GND
- added copper zone on In2.Cu, net GND
Other:
- board size 77.4 x 77.2 mm -> 86.6 x 61 mm

Commit message: f
Parts:
- added D1: RED, LED_SMD:LED_0603_1608Metric, F.Cu at (54.9, 92.7)
- added D2: RED, LED_SMD:LED_0603_1608Metric, F.Cu at (53.3, 92.7)
- added D3: RED, LED_SMD:LED_0603_1608Metric, F.Cu at (76.5, 80.0)
- added JP2: ADR0, Jumper:SolderJumper-3_P1.3mm_Bridged12_RoundedPad1.0x1.5mm_NumberLabels, F.Cu at (118.6, 82.5)
- added R33: 1K5, Resistor_SMD:R_0603_1608Metric, F.Cu at (54.9, 89.6)
- added R34: 1k, Resistor_SMD:R_0603_1608Metric, F.Cu at (53.3, 89.6)
- added R35: 1k, Resistor_SMD:R_0603_1608Metric, F.Cu at (73.5, 80.0)
- added TP10: TestPoint, TestPoint:TestPoint_Pad_1.5x1.5mm, F.Cu at (121.2, 97.2)
- added TP8: TestPoint, TestPoint:TestPoint_Pad_1.5x1.5mm, F.Cu at (65.1, 85.6)
- added TP9: TestPoint, TestPoint:TestPoint_Pad_1.5x1.5mm, F.Cu at (110.3, 67.8)
- added kibuzzard-6406DECD: G***, kibuzzard-6406DECD, F.Cu at (80.0, 82.5)
- added kibuzzard-6406DEDF: G***, kibuzzard-6406DEDF, F.Cu at (72.5, 82.5)
- added kibuzzard-6406E441: G***, kibuzzard-6406E441, F.Cu at (54.9, 95.0)
- added kibuzzard-6406E44E: G***, kibuzzard-6406E44E, F.Cu at (53.2, 95.3)
- added kibuzzard-640733B2: G***, kibuzzard-640733B2, F.Cu at (104.7, 52.9)
- moved C2 8.72 mm to (66.6, 96.8), turned to 90 degrees
- moved TP1 6.95 mm to (61.5, 100.8)
- moved H4 5.30 mm to (54.0, 101.0)
- moved H3 3.83 mm to (131.0, 101.0)
- moved FB1 1.95 mm to (56.0, 87.0)
- moved C1 1.90 mm to (60.1, 89.0), turned to 0 degrees
- moved R9 1.86 mm to (114.4, 81.1), turned to 90 degrees
- moved H2 0.87 mm to (131.0, 54.0)
- moved TP7 0.40 mm to (125.2, 87.2)
- moved R14 0.15 mm to (72.3, 95.3)
- moved C23 0.15 mm to (122.8, 72.3)
- moved C5 0.13 mm to (88.7, 96.5)
- moved RG1 0.11 mm to (115.9, 73.7)
- moved C33 0.11 mm to (92.5, 58.0)
- moved R6 0.11 mm to (121.2, 72.3)
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Connections:
- R9 pad 1: REF -> Net-(R9-Pad1)
Routing:
- net +5V: track 38.6 -> 106.1 mm, vias 0 -> 2
- net +3.3VA: track 21.8 -> 66.4 mm, vias 2 -> 6
- net Net-(C1-Pad1): track 9.89 -> 46.0 mm, vias 0 -> 2
- net VBUS: track 25.5 -> 56.4 mm, vias 0 -> 2
- net +3V3: track 169.0 -> 182.0 mm
- net /GAS_Measurements/H2_sensing: track 25.8 -> 17.4 mm, vias 0 -> 1
- net GND: track 95.9 -> 103.5 mm, vias 49 -> 253
- net Net-(R9-Pad1): track 0.00 -> 5.58 mm
- net REF: track 35.0 -> 40.5 mm
- net GPIO_9: track 0.00 -> 3.23 mm
- net /GAS_Measurements/CH4_V-gas: track 5.77 -> 7.61 mm
- net Net-(D1-Pad2): track 0.00 -> 1.45 mm
- net Net-(D2-Pad2): track 0.00 -> 1.44 mm
- net Net-(D3-Pad2): track 0.00 -> 1.44 mm
- net GPIO_5: track 77.1 -> 78.0 mm
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Other:
- board size 86.6 x 61 mm -> 85 x 55 mm
- board text added: "."
