File: HW/GMWPY/GMWPY.kicad_pcb (KiCad board)
At the start: 4 copper layers, 85 x 55 mm, 119 parts, among them J1 USB_A, J2 Conn_02x02_Odd_Even, J3 Conn_01x10, J4 Micro_SD_Card_Det, Q1 Q_PJFET_DSG, SW1 MCU_RESET, SW2 MCU_RESET, U1 AMS1117-3.3, U10 TSV991ILT, U11 TSV991ILT, U12 TSV991ILT, U13 LM4040DBZ-2.0, U14 ESP32-S3-WROOM-1, U2 SRV05-4, U3 USEQGCDACH4100, U4 TSV991ILT, U5 MCP3422, U6 TSV991ILT, U7 BME280, U8 MCP3422, U9 EC4-1000-H2

Commit message: f
Parts:
- added D4: RED, LED_SMD:LED_0603_1608Metric, F.Cu at (65.9, 82.0)
- added R36: 10k, Resistor_SMD:R_0603_1608Metric_Pad0.98x0.95mm_HandSolder, F.Cu at (85.8, 82.0)
- added R37: 10k, Resistor_SMD:R_0603_1608Metric_Pad0.98x0.95mm_HandSolder, F.Cu at (85.8, 80.4)
- added R38: 1k, Resistor_SMD:R_0603_1608Metric, F.Cu at (65.9, 80.0)
- added kibuzzard-640843D3: G***, kibuzzard-640843D3, F.Cu at (103.4, 84.4)
- added kibuzzard-640843E2: G***, kibuzzard-640843E2, F.Cu at (104.8, 80.9)
- moved TP8 2.75 mm to (66.2, 88.1)
Routing:
- net GPIO_8: track 0.00 -> 12.9 mm, vias 0 -> 2
- net GPIO_47: track 0.00 -> 6.54 mm
- net +3V3: track 182.0 -> 187.0 mm
- net GPIO_48: track 0.00 -> 4.67 mm
- net GPIO_39: track 0.00 -> 2.81 mm
- net GPIO_38: track 0.00 -> 2.69 mm
- net GPIO_37: track 0.00 -> 2.55 mm
- net GPIO_36: track 0.00 -> 2.46 mm
- net GPIO_35: track 0.00 -> 2.42 mm
- net Net-(D4-Pad2): track 0.00 -> 2.07 mm
- net GPIO_16: track 0.00 -> 2.05 mm
- net GPIO_17: track 0.00 -> 1.97 mm
- net GPIO_18: track 0.00 -> 1.96 mm
- net GPIO_46: track 0.00 -> 1.84 mm
- net GPIO_14: track 0.00 -> 1.73 mm
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- added copper zone on B.Cu, net GND

Commit message: b
Parts:
- added C35: 100n, Capacitor_SMD:C_0603_1608Metric_Pad1.08x0.95mm_HandSolder, F.Cu at (53.7, 67.0)
- added R39: 10k, Resistor_SMD:R_0603_1608Metric_Pad0.98x0.95mm_HandSolder, F.Cu at (63.5, 70.0)
- added SW3: MCU_RESET, SamacSys_Parts:PTS526SK15SMTR2LFS, F.Cu at (56.8, 61.4)
- moved kibuzzard-640733B2 1.35 mm to (103.3, 52.9)
Routing:
- net GPIO_16: track 2.05 -> 25.3 mm
- net +3V3: track 187.0 -> 189.3 mm
- net VBUS: track 56.4 -> 54.3 mm
- net GND: vias 261 -> 254
