File: HW/GMWPY/GMWPY.kicad_pcb (KiCad board)
At the start: 4 copper layers, 85 x 55 mm, 128 parts, among them J1 USB_A, J2 Conn_02x02_Odd_Even, J3 Conn_01x10, J4 Micro_SD_Card_Det, Q1 Q_PJFET_DSG, SW1 MCU_RESET, SW2 MCU_RESET, SW3 MCU_RESET, U1 AMS1117-3.3, U10 TSV991ILT, U11 TSV991ILT, U12 TSV991ILT, U13 LM4040DBZ-2.0, U14 ESP32-S3-WROOM-1, U2 SRV05-4, U3 USEQGCDACH4100, U4 TSV991ILT, U5 MCP3422, U6 TSV991ILT, U7 BME280, U8 MCP3422, U9 EC4-1000-H2

Commit message: n
Parts:
- added TP11: TestPoint, TestPoint:TestPoint_Pad_1.5x1.5mm, B.Cu at (83.3, 65.1)
- added TP12: TestPoint, TestPoint:TestPoint_Pad_1.5x1.5mm, B.Cu at (83.3, 62.5)
- added TP13: TestPoint, TestPoint:TestPoint_Pad_1.5x1.5mm, B.Cu at (78.7, 60.2)
- added kibuzzard-642169AB: G***, kibuzzard-642169AB, B.Cu at (79.9, 62.6)
- added kibuzzard-642169BA: G***, kibuzzard-642169BA, B.Cu at (79.9, 65.0)
- added kibuzzard-642169F1: G***, kibuzzard-642169F1, B.Cu at (75.0, 60.3)
Routing:
- net GPIO_44: track 2.17 -> 5.37 mm, vias 0 -> 1
- net GPIO_43: track 2.18 -> 5.10 mm, vias 0 -> 1
- net D-: track 9.08 -> 10.5 mm
- net D+: track 9.21 -> 10.6 mm
- net GND: vias 254 -> 253
